File: X19_Board_Control.kicad_sch (KiCad schematic)
At the start: 0 parts

Commit message: Progress 1
Got some symbols down, need to route things
Parts:
- added J1: Conn_01x04_Pin, symbol Connector:Conn_01x04_Pin
- added Q1, Q10, Q2, Q3, Q4, Q5, Q6, Q7, Q8, Q9: NMOS, symbol Simulation_SPICE:NMOS
- added U1: STM32C542CCT6, LQFP48-7X7, symbol board_control_manual_lib:STM32C542CCT6
- added U2: TCAN1044VDRQ1, D0008A-IPC_A, symbol board_control_manual_lib:TCAN1044VDRQ1
- added U3: BMI270, BMI270_BOS, symbol board_control_manual_lib:BMI270
- added U4: INA237AIDGSR, VSSOP_IDGSR_TEX, symbol board_control_manual_lib:INA237AIDGSR
- added U5: BNO085, LGA-28_CEV, symbol board_control_manual_lib:BNO085
- added Y1: Crystal_GND24, Crystal:Crystal_SMD_3225-4Pin_3.2x2.5mm, symbol Device:Crystal_GND24
Connections:
- new net: Y1.2 (G), Y1.4 (G)
Other:
- note added: "12 Pins (2 x 6 pins)"
- note added: "Add a USBC port so I could wire that for the STlink"
- note added: "Depth Sensor Header"
- note added: "Fade this sym, use female headers"
- note added: "USB 2.0 Connector"
