File: connector_signals.kicad_sch (KiCad schematic)
At the start: 5 parts, among them J2 Conn_01x05, J5 Conn_01x05, J6 Conn_01x05, J8 Mega Connector/Breakout (if w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, P1 USB_C_Plug_USB2.0

Commit message: Final v1
Finished making it look nice, looking for feedback
Other:
- moved on the sheet: J8

Commit message: Ok I lied v1 for real
real
Parts:
- renumbered J2 to J4, J8 to J7
Changed lines of the file:
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@@
 		(dnp no)
 		(fields_autoplaced yes)
-		(property "Reference" "#PWR028"
+		(property "Reference" "#PWR048"
 			(at 63.5 44.45 0)
 			(hide yes)
@@
 			(project "X19-Control-Board"
 				(path "/00000000-0000-0000-0000-000060e6118b/5aebb1ae-5eca-4b0a-af28-23512fd077fb"
-					(reference "#PWR028")
+					(reference "#PWR048")
 					(unit 1)
 				)
@@
 		(dnp no)
 		(fields_autoplaced yes)
-		(property "Reference" "J2"
+		(property "Reference" "J4"
 			(at 49.53 34.2899 0)
 			(show_name no)
@@
 			(project "X19-Control-Board"
 				(path "/00000000-0000-0000-0000-000060e6118b/5aebb1ae-5eca-4b0a-af28-23512fd077fb"
-					(reference "J2")
+					(reference "J4")
 					(unit 1)
 				)
@@
 		(dnp no)
 		(fields_autoplaced yes)
-		(property "Reference" "J8"
+		(property "Reference" "J7"
 			(at 194.31 19.05 0)
 			(show_name no)
@@
 			(project "X19-Control-Board"
 				(path "/00000000-0000-0000-0000-000060e6118b/5aebb1ae-5eca-4b0a-af28-23512fd077fb"
-					(reference "J8")
+					(reference "J7")
 					(unit 1)
 				)
@@
 		(dnp no)
 		(fields_autoplaced yes)
-		(property "Reference" "#PWR029"
+		(property "Reference" "#PWR049"
 			(at 101.6 45.72 0)
 			(hide yes)
@@
 			(project "X19-Control-Board"
 				(path "/00000000-0000-0000-0000-000060e6118b/5aebb1ae-5eca-4b0a-af28-23512fd077fb"
-					(reference "#PWR029")
+					(reference "#PWR049")
 					(unit 1)
 				)
@@
 		(dnp no)
 		(fields_autoplaced yes)
-		(property "Reference" "#PWR027"
+		(property "Reference" "#PWR047"
 			(at 33.02 39.37 0)
 			(hide yes)
@@
 			(project "X19-Control-Board"
 				(path "/00000000-0000-0000-0000-000060e6118b/5aebb1ae-5eca-4b0a-af28-23512fd077fb"
-					(reference "#PWR027")
+					(reference "#PWR047")
 					(unit 1)
 				)

Commit message: Rest of page feedback - Nick
Other:
- note added: "1. 5.2V and 12V nets should be the pre sense versions right? Since they're coming from power slab 2. Label CS signal CS_Pi, since it serves as the backup in case CAN fails - Nick"
- note added: "We could add this as a pin header potentially since we have a lot of space. Worst case we can make a bunch of small circular pads we can solder to - Nick"
Changed lines of the file:
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@@
+		)
+	)
+	(text "We could add this as a pin header potentially since we have a lot of space.\nWorst case we can make a bunch of small circular pads we can solder to\n\n- Nick"
+		(exclude_from_sim no)
+		(at 195.58 74.93 0)
+		(effects
+			(font
+				(size 1.27 1.27)
+				(color 255 0 0 1)
+			)
 		)
 	)
@@
 			)
 		)
+	)
+	(text "1. 5.2V and 12V nets should be\n	the pre sense versions right?\n	Since they're coming from power slab\n\n2. Label CS signal CS_Pi, since it serves\n	as the backup in case CAN fails\n\n- Nick"
+		(exclude_from_sim no)
+		(at 57.15 64.77 0)
+		(effects
+			(font
+				(size 1.27 1.27)
+				(color 255 0 0 1)
+			)
+		)
