File: connector_signals.kicad_sch (KiCad schematic)
At the start: 3 parts, among them J13 61300511821, J15 IPS1-105-01-L-D, J16 61300511821

Commit message: Sized
bang
Parts:
- removed J15: IPS1-105-01-L-D, x19_control_library:SAMTEC_IPS1-105-01-S-D, symbol Connector_Generic:Conn_02x05_Counter_Clockwise
- added J10: IPS1-105-01-L-D, x19_control_library:SAMTEC_IPS1-105-01-S-D, symbol board_control_manual_lib:IPS1-105-01-L-D
- renumbered J13 to J11, J16 to J12
Connections:
- net 12V_pre_sense: now also J10.10
- net 5.2V_pre_sense: now also J10.09
- net CAN_H: now also J10.01
- net CAN_L: now also J10.02
- net GND: now also J10.03, J10.08

Commit message: Layout Placement Is Happening
The other members are CHUD rn
Parts:
- renumbered J10 to J18, J11 to J19, J12 to J20
Changed lines of the file:
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@@
 		(dnp no)
 		(fields_autoplaced yes)
-		(property "Reference" "J10"
+		(property "Reference" "J18"
 			(at 49.53 25.4 0)
 			(show_name no)
@@
 			(project "X19-Control-Board"
 				(path "/00000000-0000-0000-0000-000060e6118b/5aebb1ae-5eca-4b0a-af28-23512fd077fb"
-					(reference "J10")
+					(reference "J18")
 					(unit 1)
 				)
@@
 		(dnp no)
 		(fields_autoplaced yes)
-		(property "Reference" "#PWR053"
+		(property "Reference" "#PWR065"
 			(at 93.98 39.37 0)
 			(hide yes)
@@
 			(project "X19-Control-Board"
 				(path "/00000000-0000-0000-0000-000060e6118b/5aebb1ae-5eca-4b0a-af28-23512fd077fb"
-					(reference "#PWR053")
+					(reference "#PWR065")
 					(unit 1)
 				)
@@
 		(dnp no)
 		(fields_autoplaced yes)
-		(property "Reference" "J11"
+		(property "Reference" "J19"
 			(at 111.76 29.2099 0)
 			(show_name no)
@@
 			(project "X19-Control-Board"
 				(path "/00000000-0000-0000-0000-000060e6118b/5aebb1ae-5eca-4b0a-af28-23512fd077fb"
-					(reference "J11")
+					(reference "J19")
 					(unit 1)
 				)
@@
 		(dnp no)
 		(fields_autoplaced yes)
-		(property "Reference" "J12"
+		(property "Reference" "J20"
 			(at 149.86 29.2099 0)
 			(show_name no)
@@
 			(project "X19-Control-Board"
 				(path "/00000000-0000-0000-0000-000060e6118b/5aebb1ae-5eca-4b0a-af28-23512fd077fb"
-					(reference "J12")
+					(reference "J20")
 					(unit 1)
 				)
@@
 		(dnp no)
 		(fields_autoplaced yes)
-		(property "Reference" "#PWR052"
+		(property "Reference" "#PWR064"
 			(at 81.28 46.99 0)
 			(hide yes)
@@
 			(project "X19-Control-Board"
 				(path "/00000000-0000-0000-0000-000060e6118b/5aebb1ae-5eca-4b0a-af28-23512fd077fb"
-					(reference "#PWR052")
+					(reference "#PWR064")
 					(unit 1)
 				)
@@
 		(dnp no)
 		(fields_autoplaced yes)
-		(property "Reference" "#PWR051"
+		(property "Reference" "#PWR063"
 			(at 27.94 41.91 0)
 			(hide yes)
@@
 			(project "X19-Control-Board"
 				(path "/00000000-0000-0000-0000-000060e6118b/5aebb1ae-5eca-4b0a-af28-23512fd077fb"
-					(reference "#PWR051")
+					(reference "#PWR063")
 					(unit 1)
 				)
