File: Sensors_Telemetry.kicad_sch (KiCad schematic)
At the start: 7 parts, among them J1 Depth_Sens_Header, J3 BN0_Side_1, J4 BN0_Side_2, U3 BMI270

Commit message: Ok I lied v1 for real
real
Parts:
- renumbered C1 to C10, C2 to C11, C16 to C12, J3 to J2, J4 to J3
Changed lines of the file:
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@@
 		(dnp no)
 		(fields_autoplaced yes)
-		(property "Reference" "C16"
+		(property "Reference" "C12"
 			(at 33.02 90.1699 0)
 			(show_name no)
@@
 			(project "X19-Control-Board"
 				(path "/00000000-0000-0000-0000-000060e6118b/a66e3e05-3f82-4c46-8531-6fdc7968dd66"
-					(reference "C16")
+					(reference "C12")
 					(unit 1)
 				)
@@
 		(dnp no)
 		(fields_autoplaced yes)
-		(property "Reference" "#PWR039"
+		(property "Reference" "#PWR032"
 			(at 93.98 63.5 0)
 			(hide yes)
@@
 			(project "X19-Control-Board"
 				(path "/00000000-0000-0000-0000-000060e6118b/a66e3e05-3f82-4c46-8531-6fdc7968dd66"
-					(reference "#PWR039")
+					(reference "#PWR032")
 					(unit 1)
 				)
@@
 		(in_pos_files yes)
 		(dnp no)
-		(property "Reference" "J4"
+		(property "Reference" "J3"
 			(at 56.134 98.552 0)
 			(show_name no)
@@
 			(project "X19-Control-Board"
 				(path "/00000000-0000-0000-0000-000060e6118b/a66e3e05-3f82-4c46-8531-6fdc7968dd66"
-					(reference "J4")
+					(reference "J3")
 					(unit 1)
 				)
@@
 		(dnp no)
 		(fields_autoplaced yes)
-		(property "Reference" "C1"
+		(property "Reference" "C10"
 			(at 34.29 46.9899 0)
 			(show_name no)
@@
 			(project "X19-Control-Board"
 				(path "/00000000-0000-0000-0000-000060e6118b/a66e3e05-3f82-4c46-8531-6fdc7968dd66"
-					(reference "C1")
+					(reference "C10")
 					(unit 1)
 				)
@@
 		(dnp no)
 		(fields_autoplaced yes)
-		(property "Reference" "#PWR042"
+		(property "Reference" "#PWR029"
 			(at 43.18 53.34 0)
 			(hide yes)
@@
 			(project "X19-Control-Board"
 				(path "/00000000-0000-0000-0000-000060e6118b/a66e3e05-3f82-4c46-8531-6fdc7968dd66"
-					(reference "#PWR042")
+					(reference "#PWR029")
 					(unit 1)
 				)
@@
 		(dnp no)
 		(fields_autoplaced yes)
-		(property "Reference" "#PWR040"
+		(property "Reference" "#PWR033"
 			(at 34.29 86.36 0)
 			(hide yes)
@@
 			(project "X19-Control-Board"
 				(path "/00000000-0000-0000-0000-000060e6118b/a66e3e05-3f82-4c46-8531-6fdc7968dd66"
-					(reference "#PWR040")
+					(reference "#PWR033")
 					(unit 1)
 				)
@@
 		(dnp no)
 		(fields_autoplaced yes)
-		(property "Reference" "C2"
+		(property "Reference" "C11"
 			(at 90.17 52.0699 0)
 			(show_name no)
@@
 			(project "X19-Control-Board"
 				(path "/00000000-0000-0000-0000-000060e6118b/a66e3e05-3f82-4c46-8531-6fdc7968dd66"
-					(reference "C2")
+					(reference "C11")
 					(unit 1)
 				)
@@
 		(dnp no)
 		(fields_autoplaced yes)
-		(property "Reference" "#PWR043"
+		(property "Reference" "#PWR030"
 			(at 46.99 55.88 0)
 			(hide yes)
@@
 			(project "X19-Control-Board"
 				(path "/00000000-0000-0000-0000-000060e6118b/a66e3e05-3f82-4c46-8531-6fdc7968dd66"
-					(reference "#PWR043")
+					(reference "#PWR030")
 					(unit 1)
 				)
@@
 		(dnp no)
 		(fields_autoplaced yes)
-		(property "Reference" "#PWR046"
+		(property "Reference" "#PWR034"
 			(at 29.21 101.6 0)
 			(hide yes)
@@
 			(project "X19-Control-Board"
 				(path "/00000000-0000-0000-0000-000060e6118b/a66e3e05-3f82-4c46-8531-6fdc7968dd66"
-					(reference "#PWR046")
+					(reference "#PWR034")
 					(unit 1)
 				)
@@
 		(in_pos_files yes)
 		(dnp no)
-		(property "Reference" "J3"
+		(property "Reference" "J2"
 			(at 58.674 82.042 0)
 			(show_name no)
@@
 			(project "X19-Control-Board"
 				(path "/00000000-0000-0000-0000-000060e6118b/a66e3e05-3f82-4c46-8531-6fdc7968dd66"
-					(reference "J3")
+					(reference "J2")
 					(unit 1)
 				)
@@
 		(dnp no)
 		(fields_autoplaced yes)
-		(property "Reference" "#PWR041"
+		(property "Reference" "#PWR031"
 			(at 30.48 58.42 0)
 			(hide yes)
@@
 			(project "X19-Control-Board"
 				(path "/00000000-0000-0000-0000-000060e6118b/a66e3e05-3f82-4c46-8531-6fdc7968dd66"
-					(reference "#PWR041")
+					(reference "#PWR031")
 					(unit 1)
 				)
@@
 		(dnp no)
 		(fields_autoplaced yes)
-		(property "Reference" "#PWR038"
+		(property "Reference" "#PWR028"
 			(at 123.19 52.07 0)
 			(hide yes)
@@
 			(project "X19-Control-Board"
 				(path "/00000000-0000-0000-0000-000060e6118b/a66e3e05-3f82-4c46-8531-6fdc7968dd66"
-					(reference "#PWR038")
-					(unit 1)
-				)
+					(reference "#PWR028")
+					(unit 1)
+				)

Commit message: Rest of page feedback - Nick
Other:
- note added: "1. ^^^^^ Delete the image, its misleading I thought it was an actual net 2. Indicate which side is which for the BNO (left / right) to help for routing and placement - Nick"
- note added: "Add note for layout to place near ROV's center of gravity as close as possible - Nick"
- note added: "Make this match the connector pinout on bluerobotics site https://bluerobotics.com/store/sensors-cameras/sensors/bar-depth-pressure-sensor/ - Nick"
Changed lines of the file:
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@@
 	(generator_version "10.0")
 	(paper "A4")
+	(text "Make this match the connector pinout on bluerobotics site\nhttps://bluerobotics.com/store/sensors-cameras/sensors/bar-depth-pressure-sensor/\n\n- Nick"
+		(exclude_from_sim no)
+		(at 149.86 57.15 0)
+		(effects
+			(font
+				(size 1.27 1.27)
+				(color 255 0 0 1)
+			)
+		)
+	)
 	(text "3V0"
 		(exclude_from_sim no)
@@
 			(font
 				(size 1.27 1.27)
+			)
+		)
+	)
+	(text "Add note for layout to place near ROV's\ncenter of gravity as close as possible\n\n- Nick"
+		(exclude_from_sim no)
+		(at 66.04 60.96 0)
+		(effects
+			(font
+				(size 1.27 1.27)
+				(color 255 0 0 1)
 			)
 		)
@@
 		)
 	)
+	(text "1. ^^^^^\n	Delete the image, its misleading \n	I thought it was an actual net\n\n2. Indicate which side is which for the BNO \n	(left / right) to help\n	for routing and placement\n\n- Nick\n"
+		(exclude_from_sim no)
+		(at 74.93 90.17 0)
+		(effects
+			(font
+				(size 1.27 1.27)
+				(color 255 0 0 1)
+			)
+			(justify left)
+		)
+	)

Commit message: add sam feedback
Other:
- note added: "you can also make a footprint for the BNO module just pretend it's an IC with a rlly weird footprint then you can have one symbol and footprint for it instead of two disjoint headers"
Changed lines of the file:
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@@
+		)
+	)
+	(text "you can also make a footprint for the BNO module\njust pretend it's an IC with a rlly weird footprint\nthen you can have one symbol and footprint for it instead of two disjoint headers"
+		(exclude_from_sim no)
+		(at 102.108 105.156 0)
+		(effects
+			(font
+				(size 1.27 1.27)
+			)
 		)
 	)
