File: Sensors_Telemetry.kicad_sch (KiCad schematic)
At the start: 7 parts, among them J18 Depth_Sens_Header, J2 BN0_Bottom_Side, J3 BN0_Top_Side_2, U3 BMI270

Commit message: 10/14
Fixing my breakout is the only thing... then we can go onto layout
Parts:
- removed C12: 0.1u, symbol Device:C
Changed lines of the file:
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@@
-	)
-	(junction
-		(at 180.34 54.61)
-		(diameter 0)
-		(color 0 0 0 0)
 	)
 	(junction
@@
 	(wire
 		(pts
-			(xy 180.34 55.88) (xy 180.34 54.61)
+			(xy 95.25 49.53) (xy 93.98 49.53)
 		)
 		(stroke
@@
 	(wire
 		(pts
-			(xy 95.25 49.53) (xy 93.98 49.53)
+			(xy 172.72 60.96) (xy 172.72 49.53)
 		)
 		(stroke
@@
 	(wire
 		(pts
-			(xy 172.72 60.96) (xy 172.72 49.53)
+			(xy 113.03 38.1) (xy 124.46 38.1)
 		)
 		(stroke
@@
 	(wire
 		(pts
-			(xy 113.03 38.1) (xy 124.46 38.1)
+			(xy 43.18 46.99) (xy 46.99 46.99)
 		)
 		(stroke
@@
 	(wire
 		(pts
-			(xy 43.18 46.99) (xy 46.99 46.99)
+			(xy 87.63 49.53) (xy 93.98 49.53)
 		)
 		(stroke
@@
 	(wire
 		(pts
-			(xy 87.63 49.53) (xy 93.98 49.53)
+			(xy 29.21 44.45) (xy 30.48 44.45)
 		)
 		(stroke
@@
 	(wire
 		(pts
-			(xy 180.34 54.61) (xy 180.34 49.53)
+			(xy 30.48 44.45) (xy 46.99 44.45)
 		)
 		(stroke
@@
 		)
 	)
-	(wire
-		(pts
-			(xy 29.21 44.45) (xy 30.48 44.45)
-		)
-		(stroke
-			(width 0)
-			(type default)
-		)
-	)
-	(wire
-		(pts
-			(xy 182.88 54.61) (xy 180.34 54.61)
-		)
-		(stroke
-			(width 0)
-			(type default)
-		)
-	)
-	(wire
-		(pts
-			(xy 30.48 44.45) (xy 46.99 44.45)
-		)
-		(stroke
-			(width 0)
-			(type default)
-		)
-	)
 	(global_label "MOSI"
 		(shape input)
@@
 	(global_label "nINT_BN0"
 		(shape input)
-		(at 182.88 54.61 0)
-		(fields_autoplaced yes)
-		(effects
-			(font
-				(size 1.27 1.27)
-			)
-			(justify left)
-		)
-		(property "Intersheetrefs" "${INTERSHEET_REFS}"
-			(at 194.6947 54.61 0)
-			(hide yes)
-			(show_name no)
-			(do_not_autoplace no)
-			(effects
-				(font
-					(size 1.27 1.27)
-				)
-				(justify left)
+		(at 180.34 49.53 270)
+		(fields_autoplaced yes)
+		(effects
+			(font
+				(size 1.27 1.27)
+			)
+			(justify right)
+		)
+		(property "Intersheetrefs" "${INTERSHEET_REFS}"
+			(at 180.34 61.3447 90)
+			(hide yes)
+			(show_name no)
+			(do_not_autoplace no)
+			(effects
+				(font
+					(size 1.27 1.27)
+				)
+				(justify right)
 			)
 		)
@@
 				(path "/00000000-0000-0000-0000-000060e6118b/a66e3e05-3f82-4c46-8531-6fdc7968dd66"
 					(reference "#PWR058")
-					(unit 1)
-				)
-			)
-		)
-	)
-	(symbol
-		(lib_id "Device:C")
-		(at 180.34 59.69 0)
-		(unit 1)
-		(body_style 1)
-		(exclude_from_sim no)
-		(in_bom yes)
-		(on_board yes)
-		(in_pos_files yes)
-		(dnp no)
-		(fields_autoplaced yes)
-		(property "Reference" "C12"
-			(at 184.15 58.4199 0)
-			(show_name no)
-			(do_not_autoplace no)
-			(effects
-				(font
-					(size 1.27 1.27)
-				)
-				(justify left)
-			)
-		)
-		(property "Value" "0.1u"
-			(at 184.15 60.9599 0)
-			(show_name no)
-			(do_not_autoplace no)
-			(effects
-				(font
-					(size 1.27 1.27)
-				)
-				(justify left)
-			)
-		)
-		(property "Footprint" ""
-			(at 181.3052 63.5 0)
-			(hide yes)
-			(show_name no)
-			(do_not_autoplace no)
-			(effects
-				(font
-					(size 1.27 1.27)
-				)
-			)
-		)
-		(property "Datasheet" ""
-			(at 180.34 59.69 0)
-			(hide yes)
-			(show_name no)
-			(do_not_autoplace no)
-			(effects
-				(font
-					(size 1.27 1.27)
-				)
-			)
-		)
-		(property "Description" "Unpolarized capacitor"
-			(at 180.34 59.69 0)
-			(hide yes)
-			(show_name no)
-			(do_not_autoplace no)
-			(effects
-				(font
-					(size 1.27 1.27)
-				)
-			)
-		)
-		(pin "1"
-		)
-		(pin "2"
-		)
-		(instances
-			(project "X19-Control-Board"
-				(path "/00000000-0000-0000-0000-000060e6118b/a66e3e05-3f82-4c46-8531-6fdc7968dd66"
-					(reference "C12")
 					(unit 1)
 				)
@@
 					(unit 1)
 				)
-			)
-		)
-	)
-	(symbol
-		(lib_id "power:GND")
-		(at 180.34 63.5 0)
-		(unit 1)
-		(body_style 1)
-		(exclude_from_sim no)
-		(in_bom yes)
-		(on_board yes)
-		(in_pos_files yes)
-		(dnp no)
-		(fields_autoplaced yes)
-		(property "Reference" "#PWR034"
-			(at 180.34 69.85 0)
-			(hide yes)
-			(show_name no)
-			(do_not_autoplace no)
-			(effects
-				(font
-					(size 1.27 1.27)
-				)
-			)
-		)
-		(property "Value" "GND"
-			(at 180.34 68.58 0)
-			(hide yes)
-			(show_name no)
-			(do_not_autoplace no)
-			(effects
-				(font
-					(size 1.27 1.27)
-				)
-			)
-		)
-		(property "Footprint" ""
-			(at 180.34 63.5 0)
-			(hide yes)
-			(show_name no)
-			(do_not_autoplace no)
-			(effects
-				(font
-					(size 1.27 1.27)
-				)
-			)
-		)
-		(property "Datasheet" ""
-			(at 180.34 63.5 0)
-			(hide yes)
-			(show_name no)
-			(do_not_autoplace no)
-			(effects
-				(font
-					(size 1.27 1.27)
-				)
-			)
-		)
-		(property "Description" "Power symbol creates a global label with name \"GND\" , ground"
-			(at 180.34 63.5 0)
-			(hide yes)
-			(show_name no)
-			(do_not_autoplace no)
-			(effects
-				(font
-					(size 1.27 1.27)
-				)
-			)
-		)
-		(pin "1"
-		)
-		(instances
-			(project "X19-Control-Board"
-				(path "/00000000-0000-0000-0000-000060e6118b/a66e3e05-3f82-4c46-8531-6fdc7968dd66"
-					(reference "#PWR034")
-					(unit 1)
-				)

Commit message: We are BACK
I am feeling myself. Lots of progress here.
Parts:
- C12: renamed from C10; footprint (none) -> Capacitor_SMD:C_0603_1608Metric_Pad1.08x0.95mm_HandSolder
- C13: renamed from C11; footprint (none) -> Capacitor_SMD:C_0603_1608Metric_Pad1.08x0.95mm_HandSolder
- J7: renamed from J18; value Depth_Sens_Header -> SM04B-GHS-TB; footprint (none) -> x19_control_library:CONN_BM04B-GHS-TBT_JST
- J8: renamed from J3; value BN0_Top_Side_2 -> 61300511821; footprint (none) -> x19_control_library:61300511821
- J9: renamed from J2; value BN0_Bottom_Side -> 61300511821; footprint (none) -> x19_control_library:61300511821
- U3: footprint BMI270_BOS -> x19_control_library:BMI270_BOS
Connections:
- net nINT_BN0 is gone; now on net INT1_BOTH_IMU: J9.6 (Pin_6)
- net INT1_BMI renamed INT1_BOTH_IMU
Other:
- note added: "BN0085"
- note removed: "Making a symbol for this next..."
Changed lines of the file:
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@@
 		)
 	)
-	(text "Making a symbol for this next..."
-		(exclude_from_sim no)
-		(at 172.466 102.616 0)
+	(text "BN0085"
+		(exclude_from_sim no)
+		(at 188.976 40.132 0)
 		(effects
 			(font
@@
 		)
 	)
-	(global_label "nINT_BN0"
+	(global_label "INT1_BOTH_IMU"
 		(shape input)
 		(at 180.34 49.53 270)
@@
 		)
 		(property "Intersheetrefs" "${INTERSHEET_REFS}"
-			(at 180.34 61.3447 90)
+			(at 180.34 66.8481 90)
 			(hide yes)
 			(show_name no)
@@
 		)
 	)
-	(global_label "INT1_BMI"
+	(global_label "CS_BN0"
+		(shape input)
+		(at 180.34 27.94 90)
+		(fields_autoplaced yes)
+		(effects
+			(font
+				(size 1.27 1.27)
+			)
+			(justify left)
+		)
+		(property "Intersheetrefs" "${INTERSHEET_REFS}"
+			(at 180.34 17.6977 90)
+			(hide yes)
+			(show_name no)
+			(do_not_autoplace no)
+			(effects
+				(font
+					(size 1.27 1.27)
+				)
+				(justify left)
+			)
+		)
+	)
+	(global_label "INT1_BOTH_IMU"
 		(shape input)
 		(at 46.99 41.91 180)
@@
 		)
 		(property "Intersheetrefs" "${INTERSHEET_REFS}"
-			(at 35.5986 41.91 0)
+			(at 29.6719 41.91 0)
 			(hide yes)
 			(show_name no)
@@
 				)
 				(justify right)
-			)
-		)
-	)
-	(global_label "CS_BN0"
-		(shape input)
-		(at 180.34 27.94 90)
-		(fields_autoplaced yes)
-		(effects
-			(font
-				(size 1.27 1.27)
-			)
-			(justify left)
-		)
-		(property "Intersheetrefs" "${INTERSHEET_REFS}"
-			(at 180.34 17.6977 90)
-			(hide yes)
-			(show_name no)
-			(do_not_autoplace no)
-			(effects
-				(font
-					(size 1.27 1.27)
-				)
-				(justify left)
 			)
 		)
@@
 		(dnp no)
 		(fields_autoplaced yes)
-		(property "Reference" "#PWR058"
+		(property "Reference" "#PWR042"
 			(at 172.72 67.31 0)
 			(hide yes)
@@
 			(project "X19-Control-Board"
 				(path "/00000000-0000-0000-0000-000060e6118b/a66e3e05-3f82-4c46-8531-6fdc7968dd66"
-					(reference "#PWR058")
+					(reference "#PWR042")
 					(unit 1)
 				)
@@
 		(dnp no)
 		(fields_autoplaced yes)
-		(property "Reference" "#PWR032"
+		(property "Reference" "#PWR040"
 			(at 93.98 63.5 0)
 			(hide yes)
@@
 			(project "X19-Control-Board"
 				(path "/00000000-0000-0000-0000-000060e6118b/a66e3e05-3f82-4c46-8531-6fdc7968dd66"
-					(reference "#PWR032")
+					(reference "#PWR040")
 					(unit 1)
 				)
@@
 		(in_pos_files yes)
 		(dnp no)
-		(property "Reference" "J3"
-			(at 173.228 40.894 90)
+		(property "Reference" "J8"
+			(at 154.94 29.972 90)
 			(show_name no)
 			(do_not_autoplace no)
@@
 			)
 		)
-		(property "Value" "BN0_Top_Side_2"
-			(at 167.132 38.354 90)
+		(property "Value" "61300511821"
+			(at 147.066 32.512 90)
 			(show_name no)
 			(do_not_autoplace no)
@@
 			)
 		)
-		(property "Footprint" ""
+		(property "Footprint" "x19_control_library:61300511821"
 			(at 172.72 33.02 0)
 			(hide yes)
@@
 			(project "X19-Control-Board"
 				(path "/00000000-0000-0000-0000-000060e6118b/a66e3e05-3f82-4c46-8531-6fdc7968dd66"
-					(reference "J3")
+					(reference "J8")
 					(unit 1)
 				)
@@
 		(dnp no)
 		(fields_autoplaced yes)
-		(property "Reference" "C10"
+		(property "Reference" "C12"
 			(at 34.29 46.9899 0)
 			(show_name no)
@@
 			)
 		)
-		(property "Footprint" ""
+		(property "Footprint" "Capacitor_SMD:C_0603_1608Metric_Pad1.08x0.95mm_HandSolder"
 			(at 31.4452 52.07 0)
 			(hide yes)
@@
 			(project "X19-Control-Board"
 				(path "/00000000-0000-0000-0000-000060e6118b/a66e3e05-3f82-4c46-8531-6fdc7968dd66"
-					(reference "C10")
+					(reference "C12")
 					(unit 1)
 				)
@@
 		(dnp no)
 		(fields_autoplaced yes)
-		(property "Reference" "#PWR029"
+		(property "Reference" "#PWR038"
 			(at 43.18 53.34 0)
 			(hide yes)
@@
 			(project "X19-Control-Board"
 				(path "/00000000-0000-0000-0000-000060e6118b/a66e3e05-3f82-4c46-8531-6fdc7968dd66"
-					(reference "#PWR029")
+					(reference "#PWR038")
 					(unit 1)
 				)
@@
 		(in_pos_files yes)
 		(dnp no)
-		(property "Reference" "J18"
+		(property "Reference" "J7"
 			(at 126.746 30.988 0)
 			(show_name no)
@@
 			)
 		)
-		(property "Value" "Depth_Sens_Header"
+		(property "Value" "SM04B-GHS-TB"
 			(at 126.238 33.782 0)
 			(show_name no)
@@
 			)
 		)
-		(property "Footprint" ""
+		(property "Footprint" "x19_control_library:CONN_BM04B-GHS-TBT_JST"
 			(at 129.54 40.64 0)
 			(hide yes)
@@
 			(project "X19-Control-Board"
 				(path "/00000000-0000-0000-0000-000060e6118b/a66e3e05-3f82-4c46-8531-6fdc7968dd66"
-					(reference "J18")
+					(reference "J7")
 					(unit 1)
 				)
@@
 		(dnp no)
 		(fields_autoplaced yes)
-		(property "Reference" "C11"
+		(property "Reference" "C13"
 			(at 90.17 52.0699 0)
 			(show_name no)
@@
 			)
 		)
-		(property "Footprint" ""
+		(property "Footprint" "Capacitor_SMD:C_0603_1608Metric_Pad1.08x0.95mm_HandSolder"
 			(at 93.0148 57.15 0)
 			(hide yes)
@@
 			(project "X19-Control-Board"
 				(path "/00000000-0000-0000-0000-000060e6118b/a66e3e05-3f82-4c46-8531-6fdc7968dd66"
-					(reference "C11")
+					(reference "C13")
 					(unit 1)
 				)
@@
 		(dnp no)
 		(fields_autoplaced yes)
-		(property "Reference" "#PWR057"
+		(property "Reference" "#PWR041"
 			(at 113.03 44.45 0)
 			(hide yes)
@@
 			(project "X19-Control-Board"
 				(path "/00000000-0000-0000-0000-000060e6118b/a66e3e05-3f82-4c46-8531-6fdc7968dd66"
-					(reference "#PWR057")
+					(reference "#PWR041")
 					(unit 1)
 				)
@@
 			)
 		)
-		(property "Footprint" "BMI270_BOS"
+		(property "Footprint" "x19_control_library:BMI270_BOS"
 			(at 46.99 34.29 0)
 			(hide yes)
@@
 		(dnp no)
 		(fields_autoplaced yes)
-		(property "Reference" "#PWR030"
+		(property "Reference" "#PWR039"
 			(at 46.99 55.88 0)
 			(hide yes)
@@
 			(project "X19-Control-Board"
 				(path "/00000000-0000-0000-0000-000060e6118b/a66e3e05-3f82-4c46-8531-6fdc7968dd66"
-					(reference "#PWR030")
+					(reference "#PWR039")
 					(unit 1)
 				)
@@
 		(in_pos_files yes)
 		(dnp no)
-		(property "Reference" "J2"
-			(at 153.416 46.228 90)
-			(show_name no)
-			(do_not_autoplace no)
-			(effects
-				(font
-					(size 1.27 1.27)
-				)
-			)
-		)
-		(property "Value" "BN0_Bottom_Side"
-			(at 154.178 48.26 90)
-			(show_name no)
-			(do_not_autoplace no)
-			(effects
-				(font
-					(size 1.27 1.27)
-				)
-			)
-		)
-		(property "Footprint" ""
+		(property "Reference" "J9"
+			(at 155.956 43.688 90)
+			(show_name no)
+			(do_not_autoplace no)
+			(effects
+				(font
+					(size 1.27 1.27)
+				)
+			)
+		)
+		(property "Value" "61300511821"
+			(at 155.956 45.974 90)
+			(show_name no)
+			(do_not_autoplace no)
+			(effects
+				(font
+					(size 1.27 1.27)
+				)
+			)
+		)
+		(property "Footprint" "x19_control_library:61300511821"
 			(at 172.72 44.45 0)
 			(hide yes)
@@
 			(project "X19-Control-Board"
 				(path "/00000000-0000-0000-0000-000060e6118b/a66e3e05-3f82-4c46-8531-6fdc7968dd66"
-					(reference "J2")
+					(reference "J9")
 					(unit 1)
 				)
@@
 		(dnp no)
 		(fields_autoplaced yes)
-		(property "Reference" "#PWR031"
+		(property "Reference" "#PWR037"
 			(at 30.48 58.42 0)
 			(hide yes)
@@
 			(project "X19-Control-Board"
 				(path "/00000000-0000-0000-0000-000060e6118b/a66e3e05-3f82-4c46-8531-6fdc7968dd66"
-					(reference "#PWR031")
+					(reference "#PWR037")
 					(unit 1)
 				)
