File: Sensors_Telemetry.kicad_sch (KiCad schematic)
At the start: 6 parts, among them J7 SM04B-GHS-TB, J8 61300511821, J9 61300511821, U3 BMI270

Commit message: Sized
bang
Parts:
- J7: footprint x19_control_library:CONN_BM04B-GHS-TBT_JST -> x19_control_library:CONN_BM04B-GHS-TBT_JST_solder_joint
- J8, J9: value 61300511821 -> 6 pin one; footprint x19_control_library:61300511821 -> Connector_PinHeader_2.54mm:PinHeader_1x06_P2.54mm_Vertical
Changed lines of the file:
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@@
 		(dnp no)
 		(fields_autoplaced yes)
-		(property "Reference" "#PWR042"
+		(property "Reference" "#PWR040"
 			(at 172.72 67.31 0)
 			(hide yes)
@@
 			(project "X19-Control-Board"
 				(path "/00000000-0000-0000-0000-000060e6118b/a66e3e05-3f82-4c46-8531-6fdc7968dd66"
-					(reference "#PWR042")
+					(reference "#PWR040")
 					(unit 1)
 				)
@@
 		(dnp no)
 		(fields_autoplaced yes)
-		(property "Reference" "#PWR040"
+		(property "Reference" "#PWR038"
 			(at 93.98 63.5 0)
 			(hide yes)
@@
 			(project "X19-Control-Board"
 				(path "/00000000-0000-0000-0000-000060e6118b/a66e3e05-3f82-4c46-8531-6fdc7968dd66"
-					(reference "#PWR040")
+					(reference "#PWR038")
 					(unit 1)
 				)
@@
 			)
 		)
-		(property "Value" "61300511821"
+		(property "Value" "6 pin one"
 			(at 147.066 32.512 90)
 			(show_name no)
@@
 			)
 		)
-		(property "Footprint" "x19_control_library:61300511821"
+		(property "Footprint" "Connector_PinHeader_2.54mm:PinHeader_1x06_P2.54mm_Vertical"
 			(at 172.72 33.02 0)
 			(hide yes)
@@
 		(dnp no)
 		(fields_autoplaced yes)
-		(property "Reference" "#PWR038"
+		(property "Reference" "#PWR036"
 			(at 43.18 53.34 0)
 			(hide yes)
@@
 			(project "X19-Control-Board"
 				(path "/00000000-0000-0000-0000-000060e6118b/a66e3e05-3f82-4c46-8531-6fdc7968dd66"
-					(reference "#PWR038")
+					(reference "#PWR036")
 					(unit 1)
 				)
@@
 			)
 		)
-		(property "Footprint" "x19_control_library:CONN_BM04B-GHS-TBT_JST"
+		(property "Footprint" "x19_control_library:CONN_BM04B-GHS-TBT_JST_solder_joint"
 			(at 129.54 40.64 0)
 			(hide yes)
@@
 		(dnp no)
 		(fields_autoplaced yes)
-		(property "Reference" "#PWR041"
+		(property "Reference" "#PWR039"
 			(at 113.03 44.45 0)
 			(hide yes)
@@
 			(project "X19-Control-Board"
 				(path "/00000000-0000-0000-0000-000060e6118b/a66e3e05-3f82-4c46-8531-6fdc7968dd66"
-					(reference "#PWR041")
+					(reference "#PWR039")
 					(unit 1)
 				)
@@
 		(dnp no)
 		(fields_autoplaced yes)
-		(property "Reference" "#PWR039"
+		(property "Reference" "#PWR037"
 			(at 46.99 55.88 0)
 			(hide yes)
@@
 			(project "X19-Control-Board"
 				(path "/00000000-0000-0000-0000-000060e6118b/a66e3e05-3f82-4c46-8531-6fdc7968dd66"
-					(reference "#PWR039")
+					(reference "#PWR037")
 					(unit 1)
 				)
@@
 			)
 		)
-		(property "Value" "61300511821"
+		(property "Value" "6 pin one"
 			(at 155.956 45.974 90)
 			(show_name no)
@@
 			)
 		)
-		(property "Footprint" "x19_control_library:61300511821"
+		(property "Footprint" "Connector_PinHeader_2.54mm:PinHeader_1x06_P2.54mm_Vertical"
 			(at 172.72 44.45 0)
 			(hide yes)
@@
 		(dnp no)
 		(fields_autoplaced yes)
-		(property "Reference" "#PWR037"
+		(property "Reference" "#PWR035"
 			(at 30.48 58.42 0)
 			(hide yes)
@@
 			(project "X19-Control-Board"
 				(path "/00000000-0000-0000-0000-000060e6118b/a66e3e05-3f82-4c46-8531-6fdc7968dd66"
-					(reference "#PWR037")
-					(unit 1)
-				)
+					(reference "#PWR035")
+					(unit 1)
+				)

Commit message: Update update 10/28
(It rhymes)
Parts:
- added J14, J15, J16, J17, J18, J19, J20, J21: Conn_01x03_Socket, symbol Connector:Conn_01x03_Socket
Connections:
- net GND: now also J14.1 (Pin_1), J15.1 (Pin_1), J16.1 (Pin_1), J17.1 (Pin_1), J18.1 (Pin_1), J19.1 (Pin_1), J20.1 (Pin_1), J21.1 (Pin_1)
- net INT1_BOTH_IMU renamed INT_BMI
- net INT_BMI: no longer J9.6 (Pin_6)
- new net INT_BN0: J9.6 (Pin_6)
- new net PWM1: J14.3 (Pin_3)
- new net PWM2: J15.3 (Pin_3)
- new net PWM3: J16.3 (Pin_3)
- new net PWM4: J17.3 (Pin_3)
- new net PWM5: J18.3 (Pin_3)
- new net PWM6: J19.3 (Pin_3)
- new net PWM7: J20.3 (Pin_3)
- new net PWM8: J21.3 (Pin_3)
- no-connect marks 7 -> 15

Commit message: Layout Placement Is Happening
The other members are CHUD rn
Parts:
- removed J8, J9: 6 pin one, Connector_PinHeader_2.54mm:PinHeader_1x06_P2.54mm_Vertical, symbol Connector:Conn_01x06_Pin
- added U7: (no value), x19_control_library:MODULE_4754, symbol board_control_manual_lib:BN0_Colin_made
- J10: renamed from J14; footprint (none) -> Connector_PinHeader_2.54mm:PinHeader_1x03_P2.54mm_Vertical
- J11: renamed from J15; footprint (none) -> Connector_PinHeader_2.54mm:PinHeader_1x03_P2.54mm_Vertical
- J12: renamed from J16; footprint (none) -> Connector_PinHeader_2.54mm:PinHeader_1x03_P2.54mm_Vertical
- J13: renamed from J17; footprint (none) -> Connector_PinHeader_2.54mm:PinHeader_1x03_P2.54mm_Vertical
- J14: renamed from J18; footprint (none) -> Connector_PinHeader_2.54mm:PinHeader_1x03_P2.54mm_Vertical
- J15: renamed from J19; footprint (none) -> Connector_PinHeader_2.54mm:PinHeader_1x03_P2.54mm_Vertical
- J16: renamed from J20; footprint (none) -> Connector_PinHeader_2.54mm:PinHeader_1x03_P2.54mm_Vertical
- J17: renamed from J21; footprint (none) -> Connector_PinHeader_2.54mm:PinHeader_1x03_P2.54mm_Vertical
- J7: footprint x19_control_library:CONN_BM04B-GHS-TBT_JST_solder_joint -> x19_control_library:vertical_CONN_BM04B-GHS-TBT_JST
- renumbered C12 to C15, C13 to C16
Connections:
- net 3.3V: now also U7.1, U7.10, U7.11
- net CS_BN0: now also U7.7
- net GND: now also U7.3
- net INT_BN0: now also U7.6
- net MISO: now also U7.5
- net MOSI: now also U7.8
- net RST_BN0: now also U7.9
- net SCLK: now also U7.4
Other:
- note removed: "3V0"
- note removed: "BN0085"
- note removed: "BT"
