File: Voltage_conv_prot.kicad_sch (KiCad schematic)
At the start: 16 parts, among them Q11 AO3400A, U4 MIC5504-3.3YM5-TR, U5 INA237AIDGSR, U6 INA237AIDGSR

Commit message: Rest of page feedback - Nick
Other:
- note added: "1. Change address lines for one of them, currently they both have same I2C address 2. U5's VBUS should be 5.2V, we trying to measure the voltage of 5.2V rail not 12V. VBUS is the voltage measurement. 3. Verify other I2C devices on ur board have different addresses. Write the address for each I2C device as a text comment next to the schematic. 4. Rename 12V_ALERT to 5.2V_ALERT for U5. I assume tha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"
- note added: "Change decoupling to 1uF as per the datasheet -Nick"
- note added: "Since we have a keyed connector to the control board we wont need this. only power slab would need it - Nick"
Changed lines of the file:
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@@
+		)
+	)
+	(text "1. Change address lines for one of them, currently they both have same I2C address\n2. U5's VBUS should be 5.2V, we trying to measure the voltage of 5.2V rail not 12V.\n	VBUS is the voltage measurement.\n3. Verify other I2C devices on ur board have different addresses. Write the address\n	for each I2C device as a text comment next to the schematic.\n4. Rename 12V_ALERT to 5.2V_ALERT for U5. I assume thats what u intended?\n5. How did you calculate shunt resistor values?\n	What current values did you use for the voltages?\n6. Set current sensing cap value to anything from 0.1uF to 1uF per the datasheet\n\n- Nick"
+		(exclude_from_sim no)
+		(at 184.15 101.6 0)
+		(effects
+			(font
+				(size 1.27 1.27)
+				(color 255 0 0 1)
+			)
 		)
 	)
@@
 			(font
 				(size 1.27 1.27)
+			)
+		)
+	)
+	(text "Change decoupling to 1uF \nas per the datasheet\n\n-Nick"
+		(exclude_from_sim no)
+		(at 58.42 54.61 0)
+		(effects
+			(font
+				(size 1.27 1.27)
+				(color 255 0 0 1)
 			)
 		)
@@
 			)
 		)
+	)
+	(text "Since we have a keyed connector to the control board\nwe wont need this. only power slab would need it\n\n- Nick"
+		(exclude_from_sim no)
+		(at 193.04 35.56 0)
+		(effects
+			(font
+				(size 1.27 1.27)
+				(color 255 0 0 1)
+			)
+		)

Commit message: add sam feedback
Other:
- note added: "would also recommend fading AO3400A is a tiny mosfet that prob can't carry enough current either, but i lowk didn't check"
Changed lines of the file:
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@@
+		)
+	)
+	(text "would also recommend fading\nAO3400A is a tiny mosfet that prob can't carry enough current either, but i lowk didn't check"
+		(exclude_from_sim no)
+		(at 213.614 45.974 0)
+		(effects
+			(font
+				(size 1.27 1.27)
+			)
 		)
 	)
