File: Voltage_conv_prot.kicad_sch (KiCad schematic)
At the start: 6 parts, among them Q1 AO3400A, U6 MIC5504-3.3YM5-TR

Commit message: Final v1
Finished making it look nice, looking for feedback
Parts:
- added C12, C13: 0.1u, symbol Device:C
- added C14, C15: C, symbol Device:C
- added R10, R8: 10k, symbol Device:R_US
- added R11: 120m, symbol Device:R_Shunt_US
- added R9: 15m, symbol Device:R_Shunt_US
- added U5, U7: INA237AIDGSR, VSSOP_IDGSR_TEX, symbol board_control_manual_lib:INA237AIDGSR
Connections:
- net 12V: now also R9.4, U5.8 (VBUS), U7.8 (VBUS)
- net 3.3V: now also C12.1, C13.1, R10.1, R8.1, U5.6 (VS), U7.6 (VS)
- net 5.2V: now also R11.4
- net GND: now also C12.2, C13.2, U5.1 (A1), U5.2 (A0), U5.7 (GND), U7.1 (A1), U7.2 (A0), U7.7 (GND)
- new net: C15.1, R11.2, U7.10 (IN+)
- new net: C15.2, R11.3, U7.9 (IN-)
- new net: C14.1, R9.2, U5.10 (IN+)
- new net: C14.2, R9.3, U5.9 (IN-)
- new net 12V_ALERT: R10.2, R8.2, U5.3 (ALERT), U7.3 (ALERT)
- new net 12V_pre_sense: R9.1
- new net 5.2V_pre_sense: R11.1
- new net SCL: U5.5 (SCL), U7.5 (SCL)
- new net SDA: U5.4 (SDA), U7.4 (SDA)
Other:
- note added: "I2C Connect"
- note added: "Power Monitoring 5.2V, 12V rails"
- note added: "R_pu"
- note added: "Reverse Polarity Protection"
- note added: "Said via"
- note added: "Said vias"
- moved on the sheet: C5, C6, D13, Q1, R32, U6

Commit message: Ok I lied v1 for real
real
Parts:
- renumbered C6 to C13, C5 to C14, C13 to C16, C14 to C17, C12 to C18, D13 to D14, Q1 to Q11, R32 to R29, R11 to R30, R10 to R31, R9 to R32, R8 to R33, U6 to U4, U7 to U5, U5 to U6
Changed lines of the file:
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@@
 		(dnp no)
 		(fields_autoplaced yes)
-		(property "Reference" "#PWR037"
+		(property "Reference" "#PWR046"
 			(at 101.6 160.02 0)
 			(hide yes)
@@
 			(project "X19-Control-Board"
 				(path "/00000000-0000-0000-0000-000060e6118b/b875d5fe-2b54-4be4-ba29-178f725d3d54"
-					(reference "#PWR037")
+					(reference "#PWR046")
 					(unit 1)
 				)
@@
 		(dnp no)
 		(fields_autoplaced yes)
-		(property "Reference" "#PWR035"
+		(property "Reference" "#PWR044"
 			(at 57.15 143.51 0)
 			(hide yes)
@@
 			(project "X19-Control-Board"
 				(path "/00000000-0000-0000-0000-000060e6118b/b875d5fe-2b54-4be4-ba29-178f725d3d54"
-					(reference "#PWR035")
+					(reference "#PWR044")
 					(unit 1)
 				)
@@
 		(dnp no)
 		(fields_autoplaced yes)
-		(property "Reference" "#PWR033"
+		(property "Reference" "#PWR042"
 			(at 101.6 119.38 0)
 			(hide yes)
@@
 			(project "X19-Control-Board"
 				(path "/00000000-0000-0000-0000-000060e6118b/b875d5fe-2b54-4be4-ba29-178f725d3d54"
-					(reference "#PWR033")
+					(reference "#PWR042")
 					(unit 1)
 				)
@@
 		(dnp no)
 		(fields_autoplaced yes)
-		(property "Reference" "C12"
+		(property "Reference" "C18"
 			(at 97.79 148.5899 0)
 			(show_name no)
@@
 			(project "X19-Control-Board"
 				(path "/00000000-0000-0000-0000-000060e6118b/b875d5fe-2b54-4be4-ba29-178f725d3d54"
-					(reference "C12")
+					(reference "C18")
 					(unit 1)
 				)
@@
 		(dnp no)
 		(fields_autoplaced yes)
-		(property "Reference" "U7"
+		(property "Reference" "U5"
 			(at 77.47 83.82 0)
 			(show_name no)
@@
 			(project "X19-Control-Board"
 				(path "/00000000-0000-0000-0000-000060e6118b/b875d5fe-2b54-4be4-ba29-178f725d3d54"
-					(reference "U7")
+					(reference "U5")
 					(unit 1)
 				)
@@
 		(dnp no)
 		(fields_autoplaced yes)
-		(property "Reference" "C13"
+		(property "Reference" "C16"
 			(at 97.79 107.9499 0)
 			(show_name no)
@@
 			(project "X19-Control-Board"
 				(path "/00000000-0000-0000-0000-000060e6118b/b875d5fe-2b54-4be4-ba29-178f725d3d54"
-					(reference "C13")
+					(reference "C16")
 					(unit 1)
 				)
@@
 		(dnp no)
 		(fields_autoplaced yes)
-		(property "Reference" "#PWR014"
+		(property "Reference" "#PWR037"
 			(at 90.17 46.99 0)
 			(hide yes)
@@
 			(project "X19-Control-Board"
 				(path "/00000000-0000-0000-0000-000060e6118b/b875d5fe-2b54-4be4-ba29-178f725d3d54"
-					(reference "#PWR014")
+					(reference "#PWR037")
 					(unit 1)
 				)
@@
 		(dnp no)
 		(fields_autoplaced yes)
-		(property "Reference" "#PWR012"
+		(property "Reference" "#PWR038"
 			(at 127 58.42 0)
 			(hide yes)
@@
 			(project "X19-Control-Board"
 				(path "/00000000-0000-0000-0000-000060e6118b/b875d5fe-2b54-4be4-ba29-178f725d3d54"
-					(reference "#PWR012")
+					(reference "#PWR038")
 					(unit 1)
 				)
@@
 		(dnp no)
 		(fields_autoplaced yes)
-		(property "Reference" "#PWR034"
+		(property "Reference" "#PWR045"
 			(at 116.8231 149.86 0)
 			(hide yes)
@@
 			(project "X19-Control-Board"
 				(path "/00000000-0000-0000-0000-000060e6118b/b875d5fe-2b54-4be4-ba29-178f725d3d54"
-					(reference "#PWR034")
+					(reference "#PWR045")
 					(unit 1)
 				)
@@
 		(dnp no)
 		(fields_autoplaced yes)
-		(property "Reference" "#PWR031"
+		(property "Reference" "#PWR039"
 			(at 57.15 100.33 0)
 			(hide yes)
@@
 			(project "X19-Control-Board"
 				(path "/00000000-0000-0000-0000-000060e6118b/b875d5fe-2b54-4be4-ba29-178f725d3d54"
-					(reference "#PWR031")
+					(reference "#PWR039")
 					(unit 1)
 				)
@@
 		(dnp no)
 		(fields_autoplaced yes)
-		(property "Reference" "R10"
+		(property "Reference" "R31"
 			(at 43.18 93.9799 0)
 			(show_name no)
@@
 			(project "X19-Control-Board"
 				(path "/00000000-0000-0000-0000-000060e6118b/b875d5fe-2b54-4be4-ba29-178f725d3d54"
-					(reference "R10")
+					(reference "R31")
 					(unit 1)
 				)
@@
 		(dnp no)
 		(fields_autoplaced yes)
-		(property "Reference" "R11"
+		(property "Reference" "R30"
 			(at 118.11 92.7099 0)
 			(show_name no)
@@
 			(project "X19-Control-Board"
 				(path "/00000000-0000-0000-0000-000060e6118b/b875d5fe-2b54-4be4-ba29-178f725d3d54"
-					(reference "R11")
+					(reference "R30")
 					(unit 1)
 				)
@@
 		(dnp no)
 		(fields_autoplaced yes)
-		(property "Reference" "#PWR015"
+		(property "Reference" "#PWR036"
 			(at 30.48 46.99 0)
 			(hide yes)
@@
 			(project "X19-Control-Board"
 				(path "/00000000-0000-0000-0000-000060e6118b/b875d5fe-2b54-4be4-ba29-178f725d3d54"
-					(reference "#PWR015")
+					(reference "#PWR036")
 					(unit 1)
 				)
@@
 		(dnp no)
 		(fields_autoplaced yes)
-		(property "Reference" "C14"
+		(property "Reference" "C17"
 			(at 104.14 133.3499 0)
 			(show_name no)
@@
 			(project "X19-Control-Board"
 				(path "/00000000-0000-0000-0000-000060e6118b/b875d5fe-2b54-4be4-ba29-178f725d3d54"
-					(reference "C14")
+					(reference "C17")
 					(unit 1)
 				)
@@
 		(dnp no)
 		(fields_autoplaced yes)
-		(property "Reference" "#PWR036"
+		(property "Reference" "#PWR043"
 			(at 57.15 140.97 0)
 			(hide yes)
@@
 			(project "X19-Control-Board"
 				(path "/00000000-0000-0000-0000-000060e6118b/b875d5fe-2b54-4be4-ba29-178f725d3d54"
-					(reference "#PWR036")
+					(reference "#PWR043")
 					(unit 1)
 				)
@@
 		(dnp no)
 		(fields_autoplaced yes)
-		(property "Reference" "U5"
+		(property "Reference" "U6"
 			(at 77.47 124.46 0)
 			(show_name no)
@@
 			(project "X19-Control-Board"
 				(path "/00000000-0000-0000-0000-000060e6118b/b875d5fe-2b54-4be4-ba29-178f725d3d54"
-					(reference "U5")
+					(reference "U6")
 					(unit 1)
 				)
@@
 		(dnp no)
 		(fields_autoplaced yes)
-		(property "Reference" "D13"
+		(property "Reference" "D14"
 			(at 151.13 46.9899 90)
 			(show_name no)
@@
 			(project "X19-Control-Board"
 				(path "/00000000-0000-0000-0000-000060e6118b/b875d5fe-2b54-4be4-ba29-178f725d3d54"
-					(reference "D13")
+					(reference "D14")
 					(unit 1)
 				)
@@
 		(dnp no)
 		(fields_autoplaced yes)
-		(property "Reference" "#PWR032"
+		(property "Reference" "#PWR041"
 			(at 114.3 109.22 0)
 			(hide yes)
@@
 			(project "X19-Control-Board"
 				(path "/00000000-0000-0000-0000-000060e6118b/b875d5fe-2b54-4be4-ba29-178f725d3d54"
-					(reference "#PWR032")
+					(reference "#PWR041")
 					(unit 1)
 				)
@@
 		(in_pos_files yes)
 		(dnp no)
-		(property "Reference" "C6"
+		(property "Reference" "C13"
 			(at 26.67 35.5599 0)
 			(show_name no)
@@
 			(project "X19-Control-Board"
 				(path "/00000000-0000-0000-0000-000060e6118b/b875d5fe-2b54-4be4-ba29-178f725d3d54"
-					(reference "C6")
+					(reference "C13")
 					(unit 1)
 				)
@@
 		(dnp no)
 		(fields_autoplaced yes)
-		(property "Reference" "R8"
+		(property "Reference" "R33"
 			(at 43.18 134.6199 0)
 			(show_name no)
@@
 			(project "X19-Control-Board"
 				(path "/00000000-0000-0000-0000-000060e6118b/b875d5fe-2b54-4be4-ba29-178f725d3d54"
-					(reference "R8")
+					(reference "R33")
 					(unit 1)
 				)
@@
 		(dnp no)
 		(fields_autoplaced yes)
-		(property "Reference" "#PWR030"
+		(property "Reference" "#PWR040"
 			(at 57.15 102.87 0)
 			(hide yes)
@@
 			(project "X19-Control-Board"
 				(path "/00000000-0000-0000-0000-000060e6118b/b875d5fe-2b54-4be4-ba29-178f725d3d54"
-					(reference "#PWR030")
+					(reference "#PWR040")
 					(unit 1)
 				)
@@
 		(in_pos_files yes)
 		(dnp no)
-		(property "Reference" "Q1"
+		(property "Reference" "Q11"
 			(at 137.16 55.88 90)
 			(show_name no)
@@
 			(project "X19-Control-Board"
 				(path "/00000000-0000-0000-0000-000060e6118b/b875d5fe-2b54-4be4-ba29-178f725d3d54"
-					(reference "Q1")
+					(reference "Q11")
 					(unit 1)
 				)
@@
 		(dnp no)
 		(fields_autoplaced yes)
-		(property "Reference" "R9"
+		(property "Reference" "R32"
 			(at 118.11 133.3499 0)
 			(show_name no)
@@
 			(project "X19-Control-Board"
 				(path "/00000000-0000-0000-0000-000060e6118b/b875d5fe-2b54-4be4-ba29-178f725d3d54"
-					(reference "R9")
+					(reference "R32")
 					(unit 1)
 				)
@@
 		(dnp no)
 		(fields_autoplaced yes)
-		(property "Reference" "R32"
+		(property "Reference" "R29"
 			(at 152.4 35.5599 0)
 			(show_name no)
@@
 			(project "X19-Control-Board"
 				(path "/00000000-0000-0000-0000-000060e6118b/b875d5fe-2b54-4be4-ba29-178f725d3d54"
-					(reference "R32")
+					(reference "R29")
 					(unit 1)
 				)
@@
 		(dnp no)
 		(fields_autoplaced yes)
-		(property "Reference" "C5"
+		(property "Reference" "C14"
 			(at 93.98 35.5599 0)
 			(show_name no)
@@
 			(project "X19-Control-Board"
 				(path "/00000000-0000-0000-0000-000060e6118b/b875d5fe-2b54-4be4-ba29-178f725d3d54"
-					(reference "C5")
+					(reference "C14")
 					(unit 1)
 				)
@@
 		(dnp no)
 		(fields_autoplaced yes)
-		(property "Reference" "#PWR013"
+		(property "Reference" "#PWR035"
 			(at 39.37 41.91 0)
 			(hide yes)
@@
 			(project "X19-Control-Board"
 				(path "/00000000-0000-0000-0000-000060e6118b/b875d5fe-2b54-4be4-ba29-178f725d3d54"
-					(reference "#PWR013")
+					(reference "#PWR035")
 					(unit 1)
 				)
@@
 		(dnp no)
 		(fields_autoplaced yes)
-		(property "Reference" "U6"
+		(property "Reference" "U4"
 			(at 59.69 22.86 0)
 			(show_name no)
@@
 			(project "X19-Control-Board"
 				(path "/00000000-0000-0000-0000-000060e6118b/b875d5fe-2b54-4be4-ba29-178f725d3d54"
-					(reference "U6")
-					(unit 1)
-				)
+					(reference "U4")
+					(unit 1)
+				)

Commit message: Commit for Milwaukee Review
Version 0.2 Completed
Parts:
- added R37: 10k, symbol Device:R_US
- C13, C14: value 0.1u -> 1u
- C15: value C -> 0.2u
- C17: value C -> 0.5u
Connections:
- net 12V: no longer R29.1, U5.8 (VBUS)
- net 12V_ALERT: no longer R31.2, U5.3 (ALERT)
- net 12V_pre_sense: now also R29.1
- net 3.3V: now also R37.1
- net 5.2V: now also U5.8 (VBUS)
- net GND: no longer U6.2 (A0)
- new net: R37.2, U6.2 (A0)
- new net 5.2V_ALERT: R31.2, U5.3 (ALERT)
Other:
- note added: "MOSFET can can take it but might not implement either"
- note removed: "Fade or keep RPP"
Changed lines of the file:
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@@
 	(text "Said via"
 		(exclude_from_sim no)
-		(at 53.34 131.318 0)
+		(at 59.944 131.318 0)
 		(effects
 			(font
@@
 		)
 	)
-	(text "I2C Connect"
-		(exclude_from_sim no)
-		(at 40.64 145.796 0)
-		(effects
-			(font
-				(size 1.27 1.27)
-			)
-		)
-	)
 	(text "Said vias"
 		(exclude_from_sim no)
@@
 		)
 	)
-	(text "Fade or keep RPP"
+	(text "MOSFET can can take it but might not implement either"
 		(exclude_from_sim no)
-		(at 140.208 26.162 0)
+		(at 139.446 64.77 0)
 		(effects
 			(font
@@
 		)
 	)
-	(text "R_pu"
-		(exclude_from_sim no)
-		(at 44.958 132.08 0)
-		(effects
-			(font
-				(size 1.27 1.27)
-			)
-		)
-	)
 	(text "Reverse Polarity Protection"
 		(exclude_from_sim no)
@@
 	(wire
 		(pts
+			(xy 49.53 134.62) (xy 57.15 134.62)
+		)
+		(stroke
+			(width 0)
+			(type default)
+		)
+	)
+	(wire
+		(pts
 			(xy 100.33 90.17) (xy 97.79 90.17)
 		)
@@
 	(wire
 		(pts
+			(xy 52.07 137.16) (xy 57.15 137.16)
+		)
+		(stroke
+			(width 0)
+			(type default)
+		)
+	)
+	(wire
+		(pts
 			(xy 100.33 138.43) (xy 113.03 138.43)
 		)
@@
 	(wire
 		(pts
+			(xy 52.07 132.08) (xy 52.07 137.16)
+		)
+		(stroke
+			(width 0)
+			(type default)
+		)
+	)
+	(wire
+		(pts
+			(xy 49.53 124.46) (xy 52.07 124.46)
+		)
+		(stroke
+			(width 0)
+			(type default)
+		)
+	)
+	(wire
+		(pts
 			(xy 120.65 140.97) (xy 115.57 140.97)
 		)
@@
 		)
 	)
+	(global_label "3.3V"
+		(shape input)
+		(at 49.53 124.46 180)
+		(fields_autoplaced yes)
+		(effects
+			(font
+				(size 1.27 1.27)
+			)
+			(justify right)
+		)
+		(property "Intersheetrefs" "${INTERSHEET_REFS}"
+			(at 42.4324 124.46 0)
+			(hide yes)
+			(show_name no)
+			(do_not_autoplace no)
+			(effects
+				(font
+					(size 1.27 1.27)
+				)
+				(justify right)
+			)
+		)
+	)
 	(global_label "12V_pre_sense"
 		(shape input)
@@
 		)
 	)
-	(global_label "12V"
+	(global_label "5.2V"
 		(shape input)
 		(at 97.79 100.33 0)
@@
 		)
 		(property "Intersheetrefs" "${INTERSHEET_REFS}"
-			(at 104.2828 100.33 0)
+			(at 104.8876 100.33 0)
 			(hide yes)
 			(show_name no)
@@
 		)
 	)
-	(global_label "12V"
+	(global_label "12V_pre_sense"
 		(shape input)
 		(at 140.97 30.48 180)
@@
 		)
 		(property "Intersheetrefs" "${INTERSHEET_REFS}"
-			(at 134.4772 30.48 0)
+			(at 124.1358 30.48 0)
 			(hide yes)
 			(show_name no)
@@
 		)
 	)
-	(global_label "12V_ALERT"
+	(global_label "5.2V_ALERT"
 		(shape input)
 		(at 38.1 99.06 180)
@@
 		)
 		(property "Intersheetrefs" "${INTERSHEET_REFS}"
-			(at 25.1363 99.06 0)
+			(at 24.5315 99.06 0)
 			(hide yes)
 			(show_name no)
@@
 	(symbol
 		(lib_id "power:GND")
-		(at 57.15 137.16 0)
-		(unit 1)
-		(body_style 1)
-		(exclude_from_sim no)
-		(in_bom yes)
-		(on_board yes)
-		(in_pos_files yes)
-		(dnp no)
-		(fields_autoplaced yes)
-		(property "Reference" "#PWR044"
-			(at 57.15 143.51 0)
-			(hide yes)
-			(show_name no)
-			(do_not_autoplace no)
-			(effects
-				(font
-					(size 1.27 1.27)
-				)
-			)
-		)
-		(property "Value" "GND"
-			(at 57.15 142.24 0)
-			(hide yes)
-			(show_name no)
-			(do_not_autoplace no)
-			(effects
-				(font
-					(size 1.27 1.27)
-				)
-			)
-		)
-		(property "Footprint" ""
-			(at 57.15 137.16 0)
-			(hide yes)
-			(show_name no)
-			(do_not_autoplace no)
-			(effects
-				(font
-					(size 1.27 1.27)
-				)
-			)
-		)
-		(property "Datasheet" ""
-			(at 57.15 137.16 0)
-			(hide yes)
-			(show_name no)
-			(do_not_autoplace no)
-			(effects
-				(font
-					(size 1.27 1.27)
-				)
-			)
-		)
-		(property "Description" "Power symbol creates a global label with name \"GND\" , ground"
-			(at 57.15 137.16 0)
-			(hide yes)
-			(show_name no)
-			(do_not_autoplace no)
-			(effects
-				(font
-					(size 1.27 1.27)
-				)
-			)
-		)
-		(pin "1"
-		)
-		(instances
-			(project "X19-Control-Board"
-				(path "/00000000-0000-0000-0000-000060e6118b/b875d5fe-2b54-4be4-ba29-178f725d3d54"
-					(reference "#PWR044")
-					(unit 1)
-				)
-			)
-		)
-	)
-	(symbol
-		(lib_id "power:GND")
 		(at 101.6 113.03 0)
 		(unit 1)
@@
 			)
 		)
-		(property "Value" "C"
+		(property "Value" "0.5u"
 			(at 104.14 135.8899 0)
 			(show_name no)
@@
 	(symbol
 		(lib_id "power:GND")
-		(at 57.15 134.62 0)
+		(at 49.53 134.62 0)
 		(unit 1)
 		(body_style 1)
@@
 		(fields_autoplaced yes)
 		(property "Reference" "#PWR043"
-			(at 57.15 140.97 0)
+			(at 49.53 140.97 0)
 			(hide yes)
 			(show_name no)
@@
 		)
 		(property "Value" "GND"
-			(at 57.15 139.7 0)
+			(at 49.53 139.7 0)
 			(hide yes)
 			(show_name no)
@@
 		)
 		(property "Footprint" ""
-			(at 57.15 134.62 0)
+			(at 49.53 134.62 0)
 			(hide yes)
 			(show_name no)
@@
 		)
 		(property "Datasheet" ""
-			(at 57.15 134.62 0)
+			(at 49.53 134.62 0)
 			(hide yes)
 			(show_name no)
@@
 		)
 		(property "Description" "Power symbol creates a global label with name \"GND\" , ground"
-			(at 57.15 134.62 0)
+			(at 49.53 134.62 0)
 			(hide yes)
 			(show_name no)
@@
 			)
 		)
-		(property "Value" "0.1u"
+		(property "Value" "1u"
 			(at 26.67 38.0999 0)
 			(show_name no)
@@
 	(symbol
 		(lib_id "Device:R_US")
+		(at 52.07 128.27 0)
+		(unit 1)
+		(body_style 1)
+		(exclude_from_sim no)
+		(in_bom yes)
+		(on_board yes)
+		(in_pos_files yes)
+		(dnp no)
+		(fields_autoplaced yes)
+		(property "Reference" "R37"
+			(at 54.61 126.9999 0)
+			(show_name no)
+			(do_not_autoplace no)
+			(effects
+				(font
+					(size 1.27 1.27)
+				)
+				(justify left)
+			)
+		)
+		(property "Value" "10k"
+			(at 54.61 129.5399 0)
+			(show_name no)
+			(do_not_autoplace no)
+			(effects
+				(font
+					(size 1.27 1.27)
+				)
+				(justify left)
+			)
+		)
+		(property "Footprint" ""
+			(at 53.086 128.524 90)
+			(hide yes)
+			(show_name no)
+			(do_not_autoplace no)
+			(effects
+				(font
+					(size 1.27 1.27)
+				)
+			)
+		)
+		(property "Datasheet" ""
+			(at 52.07 128.27 0)
+			(hide yes)
+			(show_name no)
+			(do_not_autoplace no)
+			(effects
+				(font
+					(size 1.27 1.27)
+				)
+			)
+		)
+		(property "Description" "Resistor, US symbol"
+			(at 52.07 128.27 0)
+			(hide yes)
+			(show_name no)
+			(do_not_autoplace no)
+			(effects
+				(font
+					(size 1.27 1.27)
+				)
+			)
+		)
+		(pin "1"
+		)
+		(pin "2"
+		)
+		(instances
+			(project "X19-Control-Board"
+				(path "/00000000-0000-0000-0000-000060e6118b/b875d5fe-2b54-4be4-ba29-178f725d3d54"
+					(reference "R37")
+					(unit 1)
+				)
+			)
+		)
+	)
+	(symbol
+		(lib_id "Device:R_US")
 		(at 148.59 36.83 0)
 		(unit 1)
@@
 			)
 		)
-		(property "Value" "0.1u"
+		(property "Value" "1u"
 			(at 93.98 38.0999 0)
 			(show_name no)
@@
 			)
 		)
-		(property "Value" "C"
+		(property "Value" "0.2u"
 			(at 104.14 95.2499 0)
 			(show_name no)

Commit message: Minor Edits
Just added names for some parts and reviewed with Sam
Parts:
- D14: value ???????? -> DDZ15S-7
- Q11: value AO3400A -> TSM340N06CP ROG
Other:
- note added: "Check inegrated pull down"
Changed lines of the file:
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@@
+		)
+	)
+	(text "Check inegrated pull down"
+		(exclude_from_sim no)
+		(at 49.53 119.38 0)
+		(effects
+			(font
+				(size 1.27 1.27)
+			)
 		)
 	)
@@
 	)
 	(symbol
+		(lib_id "Transistor_FET:Q_NMOS_GSD")
+		(at 137.16 49.53 90)
+		(mirror x)
+		(unit 1)
+		(body_style 1)
+		(exclude_from_sim no)
+		(in_bom yes)
+		(on_board yes)
+		(in_pos_files yes)
+		(dnp no)
+		(property "Reference" "Q11"
+			(at 137.16 55.88 90)
+			(show_name no)
+			(do_not_autoplace no)
+			(effects
+				(font
+					(size 1.27 1.27)
+				)
+			)
+		)
+		(property "Value" "TSM340N06CP ROG"
+			(at 137.16 58.42 90)
+			(show_name no)
+			(do_not_autoplace no)
+			(effects
+				(font
+					(size 1.27 1.27)
+				)
+			)
+		)
+		(property "Footprint" "Remote_Footprints:SOT-23-3L_AOS"
+			(at 134.62 54.61 0)
+			(hide yes)
+			(show_name no)
+			(do_not_autoplace no)
+			(effects
+				(font
+					(size 1.27 1.27)
+				)
+			)
+		)
+		(property "Datasheet" ""
+			(at 137.16 49.53 0)
+			(hide yes)
+			(show_name no)
+			(do_not_autoplace no)
+			(effects
+				(font
+					(size 1.27 1.27)
+				)
+			)
+		)
+		(property "Description" "N-MOSFET transistor, gate/source/drain"
+			(at 137.16 49.53 0)
+			(hide yes)
+			(show_name no)
+			(do_not_autoplace no)
+			(effects
+				(font
+					(size 1.27 1.27)
+				)
+			)
+		)
+		(pin "3"
+		)
+		(pin "1"
+		)
+		(pin "2"
+		)
+		(instances
+			(project "X19-Control-Board"
+				(path "/00000000-0000-0000-0000-000060e6118b/b875d5fe-2b54-4be4-ba29-178f725d3d54"
+					(reference "Q11")
+					(unit 1)
+				)
+			)
+		)
+	)
+	(symbol
 		(lib_id "power:GND")
 		(at 49.53 134.62 0)
@@
 			)
 		)
-		(property "Value" "????????"
+		(property "Value" "DDZ15S-7"
 			(at 151.13 49.5299 90)
 			(show_name no)
@@
 					(unit 1)
 				)
-			)
-		)
-	)
-	(symbol
-		(lib_id "Transistor_FET:Q_NMOS_GSD")
-		(at 137.16 49.53 90)
-		(mirror x)
-		(unit 1)
-		(body_style 1)
-		(exclude_from_sim no)
-		(in_bom yes)
-		(on_board yes)
-		(in_pos_files yes)
-		(dnp no)
-		(property "Reference" "Q11"
-			(at 137.16 55.88 90)
-			(show_name no)
-			(do_not_autoplace no)
-			(effects
-				(font
-					(size 1.27 1.27)
-				)
-			)
-		)
-		(property "Value" "AO3400A"
-			(at 137.16 58.42 90)
-			(show_name no)
-			(do_not_autoplace no)
-			(effects
-				(font
-					(size 1.27 1.27)
-				)
-			)
-		)
-		(property "Footprint" "Remote_Footprints:SOT-23-3L_AOS"
-			(at 134.62 54.61 0)
-			(hide yes)
-			(show_name no)
-			(do_not_autoplace no)
-			(effects
-				(font
-					(size 1.27 1.27)
-				)
-			)
-		)
-		(property "Datasheet" ""
-			(at 137.16 49.53 0)
-			(hide yes)
-			(show_name no)
-			(do_not_autoplace no)
-			(effects
-				(font
-					(size 1.27 1.27)
-				)
-			)
-		)
-		(property "Description" "N-MOSFET transistor, gate/source/drain"
-			(at 137.16 49.53 0)
-			(hide yes)
-			(show_name no)
-			(do_not_autoplace no)
-			(effects
-				(font
-					(size 1.27 1.27)
-				)
-			)
-		)
-		(pin "3"
-		)
-		(pin "1"
-		)
-		(pin "2"
-		)
-		(instances
-			(project "X19-Control-Board"
-				(path "/00000000-0000-0000-0000-000060e6118b/b875d5fe-2b54-4be4-ba29-178f725d3d54"
-					(reference "Q11")
-					(unit 1)
-				)
