File: X19-Control-Board.kicad_sch (KiCad schematic)
At the start: 17 parts, among them J1 Conn_01x04_Pin, Q1 NMOS, Q10 NMOS, Q2 NMOS, Q3 NMOS, Q4 NMOS, Q5 NMOS, Q6 NMOS, Q7 NMOS, Q8 NMOS, Q9 NMOS, U1 STM32C542CCT6, U2 TCAN1044VDRQ1, U3 BMI270, U4 INA237AIDGSR, U5 BNO085, Y1 Crystal_GND24

Commit message: Progress Commit
Aman pls save me
Parts:
- removed U5: BNO085, LGA-28_CEV, symbol board_control_manual_lib:BNO085
- added J3, J4: Conn_01x06_Pin, symbol Connector:Conn_01x06_Pin
- added U6: MIC5504-3.3YM5-TR, SOT-23-5_MC_MCH, symbol board_control_manual_lib:MIC5504-3.3YM5-TR
- added Y2: ECS-400-18-33-JGN-TR, ECS-400-18-33-JGN-TR:XTAL_ECS-400-18-33-JGN-TR, symbol board_control_manual_lib:ECS-400-18-33-JGN-TR
Connections:
- net 3.3V: now also U3.8 (VDD), J3.1 (Pin_1)
- net GND: now also U3.6 (GNDIO), U3.7 (GND), J3.3 (Pin_3)
- net SDO: now reaches U3.1 (SDO)
- net CS_BMI: now reaches U3.12 (CSB)
- net INT1_BMI: now reaches U3.4 (INT1)
- new net 3V0: J3.2 (Pin_2)
- new net BT: J4.1 (Pin_1)
- new net CS_BN0: J4.6 (Pin_6)
- new net MISO: J3.5 (Pin_5)
- new net MOSI: J4.5 (Pin_5)
- new net RST_BN0: J4.4 (Pin_4)
- new net SCLK: J3.4 (Pin_4)
- new net VDD: J4.2 (Pin_2), J4.3 (Pin_3)
- new net nINT_BN0: J3.6 (Pin_6)
- no-connect marks 0 -> 5
Other:
- note added: "Need a TVS diode/array"
- note removed: "12 Pins (2 x 6 pins)"
- note removed: "Fade this sym, use female headers"
- moved on the sheet: U1, U2, U3, U4

Commit message: Mid-day Push
Progress later
Parts:
- removed Q1, Q10, Q2, Q3, Q4, Q5, Q6, Q7, Q8, Q9: NMOS, symbol Simulation_SPICE:NMOS
- removed U4: INA237AIDGSR, VSSOP_IDGSR_TEX, symbol board_control_manual_lib:INA237AIDGSR
- removed Y1: Crystal_GND24, Crystal:Crystal_SMD_3225-4Pin_3.2x2.5mm, symbol Device:Crystal_GND24
- added C1, C11, C12, C13, C2, C5, C6, C7, C9: 0.1u, symbol Device:C
- added C10, C14, C15, C3, C4, C8: C, symbol Device:C
- added D1, D2: LED, symbol Device:LED
- added R1, R2, R3, R5, R6: R_US, symbol Device:R_US
- added R10, R8: 10k, symbol Device:R_US
- added R11: 120m, symbol Device:R_Shunt_US
- added R4, R7: 60, symbol Device:R_US
- added R9: 15m, symbol Device:R_Shunt_US
- added U5, U7: INA237AIDGSR, VSSOP_IDGSR_TEX, symbol board_control_manual_lib:INA237AIDGSR
- J1: value Conn_01x04_Pin -> Depth_Sens_Header
Connections:
- net SDO is gone; now on net MISO: U3.1 (SDO)
- net 3.3V: now also J1.1 (Pin_1), U1.24 (VDD), U1.47 (VSS), U3.5 (VDDIO), U6.5 (VOUT), C1.1, C10.1, C12.1, C13.1, C2.1, C5.1, C7.1, C8.1, C9.1, D2.2 (A), R10.1, R8.1, U5.6 (VS), U7.6 (VS)
- net 5.2V: now also U6.1 (VIN), U6.3 (EN), C6.1, D1.2 (A), R11.4
- net GND: now also J1.4 (Pin_4), U1.23 (VSS), U1.48 (VDD), U2.2 (GND), U6.2 (GND), C1.2, C10.2, C12.2, C13.2, C2.2, C5.2, C6.2, C7.2, C8.2, C9.2, R2.2, R3.2, U5.1 (A1), U5.2 (A0), U5.7 (GND), U7.1 (A1), U7.2 (A0), U7.7 (GND)
- net MOSI: now also U3.14 (SDX)
- net SCLK: now also U3.13 (SCX)
- net at U2.6 (CANL): now also R7.2
- net at U2.7 (CANH): now also R4.1
- net SDA: now reaches J1.2 (Pin_2)
- net SDA: now also U5.4 (SDA), U7.4 (SDA)
- net SCL: now reaches J1.3 (Pin_3)
- net SCL: now also U5.5 (SCL), U7.5 (SCL)
- new net: D2.1 (K), R3.1
- new net: C14.1, R9.2, U5.10 (IN+)
- new net: C14.2, R9.3, U5.9 (IN-)
- new net: C15.1, R11.2, U7.10 (IN+)
- new net: C15.2, R11.3, U7.9 (IN-)
- new net: C11.1, R4.2, R7.1
- new net: D1.1 (K), R2.1
- new net 12V: R9.4, U5.8 (VBUS), U7.8 (VBUS)
- new net 12V_ALERT: R10.2, R8.2, U5.3 (ALERT), U7.3 (ALERT)
- new net 12V_pre_sense: R9.1
- new net 5.2V_pre_sense: R11.1
- no-connect marks 5 -> 7
Other:
- added sheet MOSFET_driver (untitled.kicad_sch)
- note added: "ADC? (Prob no)"
- note added: "Can-specific TVS diode"
- note added: "Damping resistor, input capacitance for this external oscillator"
- note added: "GPIO"
- note added: "I2C"
- note added: "I2C Connect"
- note added: "I2C Pullups"
- note added: "PWM"
- note added: "R_pu"
- note added: "Said via"
- note added: "What val"
- moved on the sheet: J1, J3, J4, Y2

Commit message: Much more progress
hi mom
Parts:
- removed C1, C12, C13, C2, C5, C6, C9: 0.1u, symbol Device:C
- removed C14, C15: C, symbol Device:C
- removed J1: Depth_Sens_Header, symbol Connector:Conn_01x04_Pin
- removed J3, J4: Conn_01x06_Pin, symbol Connector:Conn_01x06_Pin
- removed R10, R8: 10k, symbol Device:R_US
- removed R11: 120m, symbol Device:R_Shunt_US
- removed R9: 15m, symbol Device:R_Shunt_US
- removed U3: BMI270, BMI270_BOS, symbol board_control_manual_lib:BMI270
- removed U5, U7: INA237AIDGSR, VSSOP_IDGSR_TEX, symbol board_control_manual_lib:INA237AIDGSR
- removed U6: MIC5504-3.3YM5-TR, SOT-23-5_MC_MCH, symbol board_control_manual_lib:MIC5504-3.3YM5-TR
- added C17, C18, C20: 0.1u, symbol Device:C
- added CR1: ESD2CAN24DBZRQ1, SOT-23_DBZ_TEX, symbol board_control_manual_lib:ESD2CAN24DBZRQ1
- added D15: LED, symbol Device:LED
- added R34: R_US, symbol Device:R_US
- added TP1: 12V_TP, symbol Connector:TestPoint
- added TP2: 5.2V_TP, symbol Connector:TestPoint
- added TP3: 3.3VTP, symbol Connector:TestPoint
- added TP4: GND_TP, symbol Connector:TestPoint
- C10: value C -> 0.1u
- C3, C4: value C -> 27p
- C8: value C -> 4.7u
- R1: value R_US -> 0
- R5, R6: value R_US -> 10k
Connections:
- net 12V: now also D15.2 (A), TP1.1
- net 3.3V: now also C10.2, R5.1, R6.1, U1.36 (VDD), U1.48 (VDD), U2.5 (VIO), C17.1, TP3.1; no longer C10.1, U1.47 (VSS)
- net 5.2V: now also U2.3 (VCC), C18.1, TP2.1
- net CS_BMI: now also U1.31 (PA10)
- net GATE1: now also U1.10 (PA0)
- net GATE10: now also U1.22 (VCAP)
- net GATE2: now also U1.11 (PA1)
- net GATE3: now also U1.12 (PA2)
- net GATE4: now also U1.13 (PA3)
- net GATE5: now also U1.17 (PA7)
- net GATE6: now also U1.18 (PB0)
- net GATE7: now also U1.19 (PB1)
- net GATE8: now also U1.20 (PB2)
- net GATE9: now also U1.21 (PB10)
- net GND: now also C10.1, C11.2, C3.2, C4.2, U1.35 (VSS), U1.47 (VSS), Y2.2 (GND), C17.2, C18.2, C20.1, CR1.3, R34.2, TP4.1; no longer C10.2, U1.48 (VDD)
- net INT1_BMI: now also U1.25 (PB12)
- net MISO: now also U1.16 (PA6)
- net MOSI: now also U1.14 (PA4)
- net PWM_A1: now also U1.46 (PB9)
- net PWM_A2: now also U1.45 (PB8)
- net PWM_B1: now also U1.44 (PH2-BOOT0)
- net PWM_B2: now also U1.43 (PB7)
- net PWM_C1: now also U1.42 (PB6)
- net PWM_C2: now also U1.41 (PB5)
- net PWM_D1: now also U1.40 (PB4)
- net PWM_D2: now also U1.39 (PB3)
- net RST_BN0: now also U1.26 (PB13)
- net SCL: now also R5.2, U1.32 (PA11)
- net SCLK: now also U1.15 (PA5)
- net SDA: now also R6.2, U1.33 (PA12)
- net nINT_BN0: now also U1.27 (PB14)
- net STM_TO_INPUT_CAN: now reaches U2.1 (TXD)
- net STM_TO_INPUT_CAN: now also U1.29 (PA8)
- net STM_TO_OUTPUT_CAN: now reaches U2.4 (RXD)
- net STM_TO_OUTPUT_CAN: now also U1.28 (PB15)
- net at R7.2, U2.6 (CANL): now also CR1.2
- net at R4.1, U2.7 (CANH): now also CR1.1
- net OSC_IN: now reaches C4.1
- net OSC_IN: now also C3.1, R1.1, U1.5 (PH0-OSC_IN)
- net at R1.2: now also Y2.1 (IN/OUT)
- net SWDIO: now reaches U1.34 (PA13)
- net SWCLK: now reaches U1.37 (PA14)
- net OSC_OUT: now reaches U1.6 (PH1-OSC_OUT)
- net OSC_OUT: now also Y2.3 (OUT/IN)
- net nRST: now reaches U1.7 (NRST)
- net nRST: now also C20.2
- new net: D15.1 (K), R34.1
- no-connect marks 7 -> 3
Other:
- added sheet Connector_Signals (connector_signals.kicad_sch)
- added sheet Power_Monitoring (Power_Monitoring.kicad_sch)
- added sheet Sensors_Telemetry (Sensors_Telemetry.kicad_sch)
- added sheet Voltage Conv-Protec (Voltage_conv_prot.kicad_sch)
- note added: "Do we need?"
- note added: "Low current/freq playa"
- note added: "Not using DAC/ADC GND VREF+?"
- note added: "PWM (Bitbang GPIO)"
- note added: "They didn't specify one?"
- note removed: "Add a USBC port so I could wire that for the STlink"
- note removed: "Can-specific TVS diode"
- note removed: "Depth Sensor Header"
- note removed: "I2C"
- note removed: "I2C Connect"
- note removed: "I2C Pullups"
- note removed: "Need a TVS diode/array"
- note removed: "PWM"
- note removed: "R_pu"
- note removed: "Said via"
- note removed: "USB 2.0 Connector"
- moved on the sheet: C10, C11, C3, C4, C7, C8, R1, R4, R5, R6, R7, U1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

Commit message: Final v1
Finished making it look nice, looking for feedback
Other:
- sheet Voltage Conv-Protec renamed Voltage Conv-Protec-Monitoring
- removed sheet Power_Monitoring
- note added: "CAN Transceiver"
- note added: "Categorized Designs"
- note added: "Crystal Oscillator"
- note added: "MCU Connections"
- note added: "Test Points, LEDs"
- note removed: "Damping resistor, input capacitance for this external oscillator"
- moved on the sheet: C11, C18, C3, C4, CR1, D1, D15, D2, R1, R2, R3, R34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

Commit message: Ok I lied v1 for real
real
Parts:
- renumbered C10 to C1, C20 to C2, C17 to C3, C7 to C4, C8 to C5, C3 to C6, C4 to C7, C18 to C8, C11 to C9, D15 to D1, D1 to D2, D2 to D3, R5 to R1, R6 to R2, R1 to R3, R34 to R4, R2 to R5, R3 to R6, R4 to R7, R7 to R8, TP4 to TP2, TP2 to TP3, TP3 to TP4, Y2 to Y1

Commit message: Nick Initial Feedback - Page 1
Other:
- note added: "100nF Bypass cap for VIO -Nick"
- note added: "<-Tie to Ground -Nick"
- note added: "General: - testpoints and debugging: - break out CAN signals to a header for debugging - break out SPI -"
- note added: "MCU: - add debug LED to STM GPIO - break out a few GPIO STM pins to a pin header - why do gpio bitbang for PWM? Cant we just use the STM's timer channels? - add no connect (NC) to the unused STM pins"
- note added: "Place TVS close to connector -Nick"
- note added: "Resistor Values? - Nick"
- note removed: "Do we need?"
Changed lines of the file:
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@@
+		)
+	)
+	(text "Resistor Values? - Nick"
+		(exclude_from_sim no)
+		(at 269.24 111.76 0)
+		(effects
+			(font
+				(size 1.27 1.27)
+				(color 255 0 0 1)
+			)
+		)
+	)
+	(text "General:\n- testpoints and debugging:\n	- break out CAN signals to a header for debugging\n	- break out SPI\n	- "
+		(exclude_from_sim no)
+		(at 114.3 124.46 0)
+		(effects
+			(font
+				(size 1.27 1.27)
+				(color 255 0 0 1)
+			)
+			(justify left)
 		)
 	)
@@
 				(size 1.27 1.27)
 			)
+		)
+	)
+	(text "MCU:\n- add debug LED to STM GPIO\n- break out a few GPIO STM pins to a pin header\n- why do gpio bitbang for PWM? Cant we just use the STM's timer channels?\n- add no connect (NC) to the unused STM pins"
+		(exclude_from_sim no)
+		(at 114.3 107.95 0)
+		(effects
+			(font
+				(size 1.27 1.27)
+				(color 255 0 0 1)
+			)
+			(justify left)
+		)
+	)
+	(text "100nF Bypass cap \nfor VIO -Nick"
+		(exclude_from_sim no)
+		(at 72.39 158.75 0)
+		(effects
+			(font
+				(size 1.27 1.27)
+				(color 255 0 0 1)
+			)
+			(justify left)
 		)
 	)
@@
 		)
 	)
-	(text "Do we need?"
+	(text "Place TVS close \nto connector -Nick"
 		(exclude_from_sim no)
-		(at 78.486 169.164 0)
+		(at 148.59 167.64 0)
 		(effects
 			(font
@@
 			)
 		)
+	)
+	(text "<-Tie to Ground -Nick"
+		(exclude_from_sim no)
+		(at 82.55 168.91 0)
+		(effects
+			(font
+				(size 1.27 1.27)
+				(color 255 0 0 1)
+			)
+		)

Commit message: Rest of page feedback - Nick
Other:
- note added: "General: - testpoints and debugging: - break out CAN signals to a header for debugging (2.54mm male pin header) - break out SPI (SPI data lines as well as CS_PI) - same header as CAN (2.54mm male pin header) - add no connect X to unused pins - fill unknown passive values (caps, resistors)"
- note removed: "General: - testpoints and debugging: - break out CAN signals to a header for debugging - break out SPI -"
Changed lines of the file:
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@@
 		)
 	)
-	(text "General:\n- testpoints and debugging:\n	- break out CAN signals to a header for debugging\n	- break out SPI\n	- "
+	(text "General:\n- testpoints and debugging:\n	- break out CAN signals to a header for debugging (2.54mm male pin header)\n	- break out SPI (SPI data lines as well as CS_PI)\n		- same header as CAN (2.54mm male pin header)\n\n- add no connect X to unused pins\n- fill unknown passive values (caps, resistors)\n"
 		(exclude_from_sim no)
 		(at 114.3 124.46 0)

Commit message: add sam feedback
Other:
- note added: "10k pullups are a lil weak for i2c they will work but 4k7 is typ"
- note added: "load caps should be one on each output pin, not both on one"
- note added: "they usually won't it's implied to use decoupling on ICs"
Changed lines of the file:
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@@
+		)
+	)
+	(text "they usually won't\nit's implied to use decoupling on ICs"
+		(exclude_from_sim no)
+		(at 38.1 146.05 0)
+		(effects
+			(font
+				(size 1.27 1.27)
+			)
 		)
 	)
@@
 		)
 	)
+	(text "10k pullups are a lil weak for i2c\nthey will work but 4k7 is typ"
+		(exclude_from_sim no)
+		(at 165.354 54.102 0)
+		(effects
+			(font
+				(size 1.27 1.27)
+			)
+		)
+	)
 	(text "What val"
 		(exclude_from_sim no)
@@
 		(effects
 			(font
+				(size 1.27 1.27)
+			)
+		)
+	)
+	(text "load caps should be one on each output pin, not both on one"
+		(exclude_from_sim no)
+		(at 65.786 131.572 0)
+		(effects
+			(font
