File: X19-Control-Board.kicad_sch (KiCad schematic)
At the start: 31 parts, among them U1 STM32C542CCT6, U2 TCAN1044VDRQ1, Y1 ECS-400-18-33-JGN-TR

Commit message: 10/14
Fixing my breakout is the only thing... then we can go onto layout
Parts:
- removed Y1: ECS-400-18-33-JGN-TR, ECS-400-18-33-JGN-TR:XTAL_ECS-400-18-33-JGN-TR, symbol board_control_manual_lib:ECS-400-18-33-JGN-TR
- added C20: 2.2u, symbol Device:C
- added R29: 10k, symbol Device:R_US
- added Y2: ECS-240-8-37B-CKY-TR, symbol Device:Crystal_GND24
- C6, C7: value 27p -> 8p
- R34: value 65 -> 220
Connections:
- net +3.3V: now also U1.22 (VCAP), C20.1
- net GATE10: now also U1.1 (PE2); no longer U1.22 (VCAP)
- net GND: now also U1.8 (VREF-), U1.9 (VREF+), C20.2, Y2.2 (G), Y2.4 (G)
- net OSC_IN: now also C6.1, Y2.1; no longer R3.1
- net OSC_OUT: now also R3.2; no longer C7.1
- net PWM_A1: now also U1.29 (PA8); no longer U1.46 (PB9)
- net PWM_A2: no longer U1.45 (PB8)
- net PWM_B1: now also U1.28 (PB15); no longer U1.44 (PH2-BOOT0)
- net STM_TO_INPUT_CAN: now also U1.46 (PB9); no longer U1.29 (PA8)
- net STM_TO_OUTPUT_CAN: now also U1.45 (PB8); no longer U1.28 (PB15)
- net CS_BN0: now reaches U1.38 (PA15)
- net MISO renamed PI_MISO
- net MOSI renamed PI_MOSI
- new net: C7.1, R3.1, Y2.3
- no-connect marks 7 -> 3
Other:
- added sheet temp_idea_555 (temp_idea_555.kicad_sch)
- note added: "ECS-240-8-37B-CKY-TR ADD THIS INSTEAD FOR CRYSTAl"
- note added: "NEW CAP VALUES"
- note added: "We can only maybe add to the BOOT0"
- moved on the sheet: C1, C6, C7

Commit message: We are BACK
I am feeling myself. Lots of progress here.
Parts:
- removed C3: 0.1u, symbol Device:C
- removed R1, R2, R29: 10k, symbol Device:R_US
- added C11: 0.1u, Capacitor_SMD:C_0603_1608Metric_Pad1.08x0.95mm_HandSolder, symbol Device:C
- added R37, R5, R6: 10k, Resistor_SMD:R_0603_1608Metric_Pad0.98x0.95mm_HandSolder, symbol Device:R_US
- C1: renamed from C20; footprint (none) -> Capacitor_SMD:C_0603_1608Metric_Pad1.08x0.95mm_HandSolder
- C10: renamed from C1; footprint (none) -> Capacitor_SMD:C_0603_1608Metric_Pad1.08x0.95mm_HandSolder
- C2: renamed from C19; footprint (none) -> Capacitor_SMD:C_0603_1608Metric_Pad1.08x0.95mm_HandSolder
- C3: renamed from C8; footprint (none) -> Capacitor_SMD:C_0603_1608Metric_Pad1.08x0.95mm_HandSolder
- C4: renamed from C2; footprint (none) -> Capacitor_SMD:C_0603_1608Metric_Pad1.08x0.95mm_HandSolder
- C5: renamed from C4; footprint (none) -> Capacitor_SMD:C_0603_1608Metric_Pad1.08x0.95mm_HandSolder
- C6: renamed from C5; footprint (none) -> Capacitor_SMD:C_0603_1608Metric_Pad1.08x0.95mm_HandSolder
- C7: renamed from C6; footprint (none) -> Capacitor_SMD:C_0603_1608Metric_Pad1.08x0.95mm_HandSolder
- C8: renamed from C7; footprint (none) -> Capacitor_SMD:C_0603_1608Metric_Pad1.08x0.95mm_HandSolder
- C9: footprint (none) -> Capacitor_SMD:C_0603_1608Metric_Pad1.08x0.95mm_HandSolder
- CR1: footprint SOT-23_DBZ_TEX -> x19_control_library:ESD2CAN24DBZRQ1
- D1: renamed from D15; value RED -> ORANGE; footprint (none) -> x19_control_library:LTST-C191KFKT
- D2: renamed from D1; footprint (none) -> x19_control_library:LTST-C191KFKT
- D3: renamed from D2; footprint (none) -> x19_control_library:LTST-C191KFKT
- D4: renamed from D3; footprint (none) -> x19_control_library:LTST-C191KFKT
- R1: renamed from R3; footprint (none) -> Resistor_SMD:R_0603_1608Metric_Pad0.98x0.95mm_HandSolder
- R10: renamed from R6; value 65 -> 120; footprint (none) -> Resistor_SMD:R_0603_1608Metric_Pad0.98x0.95mm_HandSolder
- R2: renamed from R7; footprint (none) -> Resistor_SMD:R_0603_1608Metric_Pad0.98x0.95mm_HandSolder
- R3: renamed from R8; footprint (none) -> Resistor_SMD:R_0603_1608Metric_Pad0.98x0.95mm_HandSolder
- R7: renamed from R34; value 220 -> 120; footprint (none) -> Resistor_SMD:R_0603_1608Metric_Pad0.98x0.95mm_HandSolder
- R8: renamed from R4; value 440 -> 1k; footprint (none) -> Resistor_SMD:R_0603_1608Metric_Pad0.98x0.95mm_HandSolder
- R9: renamed from R5; value 310 -> 120; footprint (none) -> Resistor_SMD:R_0603_1608Metric_Pad0.98x0.95mm_HandSolder
- TP1: renamed from TP2; footprint (none) -> TestPoint:TestPoint_Pad_D3.0mm
- TP2: renamed from TP3; footprint (none) -> TestPoint:TestPoint_Pad_D3.0mm
- TP3: renamed from TP1; footprint (none) -> TestPoint:TestPoint_Pad_D3.0mm
- TP4: footprint (none) -> TestPoint:TestPoint_Pad_D3.0mm
- U1: renamed from U2; value TCAN1044VDRQ1 -> TCAN1044AEVDRQ1; footprint D0008A-IPC_A -> x19_control_library:TCAN1044AEVDRQ1
- U2: renamed from U1; footprint LQFP48-7X7 -> x19_control_library:STM32C542CCT6
- Y1: renamed from Y2; footprint (none) -> x19_control_library:ECS-240-8-37CKM_ECS
Connections:
- net GATE10 is gone; now on net RST_BN0: U2.1 (PE2)
- net GATE9 is gone; now on net SCL: U2.21 (PB10)
- net PWM_B2 is gone; now on net STM_TO_OUTPUT_CAN: U2.43 (PB7)
- net PWM_C1 is gone; now on net CS_BN0: U2.42 (PB6)
- net PWM_C2 is gone; now on net CS_BMI: U2.41 (PB5)
- net CS_BMI: no longer U2.31 (PA10)
- net CS_BN0: no longer U2.38 (PA15)
- net DEBUG: now also U2.46 (PB9); no longer U2.30 (PA9)
- net GND: now also C11.1
- net RST_BN0: no longer U2.26 (PB13)
- net SCL: now also R5.2; no longer U2.32 (PA11)
- net SDA: now also R6.2
- net STM_TO_INPUT_CAN: now also U2.45 (PB8); no longer U2.46 (PB9)
- net STM_TO_OUTPUT_CAN: no longer U2.45 (PB8)
- net +12V renamed 12V
- net +3.3V renamed 3.3V
- net 3.3V: now also C11.2, R37.1, R5.1, R6.1
- net +5.2V renamed 5.2V
- net GATE1 renamed PWM1
- net GATE2 renamed PWM2
- net GATE3 renamed PWM3
- net GATE4 renamed PWM4
- net GATE5 renamed SOL1A
- net GATE6 renamed SOL1B
- net GATE7 renamed SOL2A
- net GATE8 renamed SOL2B
- net INT1_BMI renamed SOL5B
- net PI_MISO renamed MISO
- net PI_MOSI renamed MOSI
- net PWM_A1 renamed PWM5
- net PWM_B1 renamed SOL4A
- net PWM_D1 renamed INT1_BOTH_IMU
- net PWM_D2 renamed SOL3A
- net nINT_BN0 renamed SOL4B
- new net PWM6: U2.30 (PA9)
- new net PWM7: U2.31 (PA10)
- new net PWM8: U2.32 (PA11)
- new net SOL3B: U2.38 (PA15)
- new net SOL5A: U2.26 (PB13)
- no-connect marks 3 -> 4
Other:
- removed sheet temp_idea_555
- note added: "* Assuming no ADC"
- note added: "10mA all"
- note added: "Check TX and RX pins for CANFD"
- note added: "Configured as push pull right now"
- note added: "NEW CAP VALUES?"
- note added: "Open drain? Would need a pull up if so"
- note added: "Place TVS close to connector"
- note added: "crystal 3225 gnd 24"
- note removed: "- break out a few GPIO STM pins to a pin header"
- note removed: "20mA for Blue (3.3V), Red (2.0V) 10mA for Green (2.1V)"
- note removed: "ADC? (Prob no)"
- note removed: "Add LED debug"
- note removed: "ECS-240-8-37B-CKY-TR ADD THIS INSTEAD FOR CRYSTAl"
- note removed: "GPIO"
- note removed: "Layout Notes"
- note removed: "NEW CAP VALUES"
- note removed: "PWM (Bitbang GPIO)"
- note removed: "Place TVS close to connector -Nick"
- note removed: "Unvisited Questions:"
- note removed: "We can only maybe add to the BOOT0"
- note removed: "alert pins from the power monitoring"
- moved on the sheet: C4, D2, R8
