File: X19-Control-Board.kicad_sch (KiCad schematic)
At the start: 33 parts, among them U1 TCAN1044AEVDRQ1, U2 STM32C542CCT6, Y1 ECS-240-8-37B-CKY-TR

Commit message: Sized
bang
Parts:
- removed R37: 10k, Resistor_SMD:R_0603_1608Metric_Pad0.98x0.95mm_HandSolder, symbol Device:R_US
- D1, D2, D3, D4: footprint x19_control_library:LTST-C191KFKT -> x19_control_library:LTST-C191KFKT_1_anode_2_cathode
- renumbered C11 to C10, C10 to C11, C4 to C2, C2 to C3, C3 to C4, R5 to R1, R1 to R2, R2 to R3, R3 to R4, R6 to R5, R7 to R6, R8 to R7, R9 to R8, R10 to R9

Commit message: Update update 10/28
(It rhymes)
Parts:
- added C18, C19, C20: 22u, Capacitor_SMD:C_0603_1608Metric_Pad1.08x0.95mm_HandSolder, symbol Device:C
- added R32: 10k, Resistor_SMD:R_0603_1608Metric_Pad0.98x0.95mm_HandSolder, symbol Device:R_US
Connections:
- net 12V: now also C18.1, C19.1
- net 3.3V: no longer C1.1, U2.22 (VCAP)
- net 5.2V: now also C20.1
- net GND: now also C18.2, C19.2, C20.2, R32.2
- net INT_BN0: now reaches U2.2 (PC13)
- net at U2.44 (PH2-BOOT0): now also R32.1
- net INT1_BOTH_IMU renamed INT_BMI
- net STM_TO_INPUT_CAN renamed CAN_RX
- net CAN_RX: now also U1.4 (RXD); no longer U1.1 (TXD)
- net STM_TO_OUTPUT_CAN renamed CAN_TX
- net CAN_TX: now also U1.1 (TXD); no longer U1.4 (RXD)
- new net: C1.1, U2.22 (VCAP)
- no-connect marks 4 -> 2
Other:
- note added: "1206 package size"
- note added: "Footprint fix, it's backwand"
- note removed: "Configured as push pull right now"
- note removed: "Open drain? Would need a pull up if so"

Commit message: Layout Placement Is Happening
The other members are CHUD rn
Parts:
- C12: renamed from C20; footprint Capacitor_SMD:C_0603_1608Metric_Pad1.08x0.95mm_HandSolder -> Capacitor_SMD:C_1206_3216Metric_Pad1.33x1.80mm_HandSolder
- C13: renamed from C18; footprint Capacitor_SMD:C_0603_1608Metric_Pad1.08x0.95mm_HandSolder -> Capacitor_SMD:C_1206_3216Metric_Pad1.33x1.80mm_HandSolder
- C14: renamed from C19; footprint Capacitor_SMD:C_0603_1608Metric_Pad1.08x0.95mm_HandSolder -> Capacitor_SMD:C_1206_3216Metric_Pad1.33x1.80mm_HandSolder
- renumbered R9 to R10, R32 to R5, R5 to R6, R6 to R7, R7 to R8, R8 to R9
Other:
- moved on the sheet: C12, C13, C14
