File: untitled.kicad_sch (KiCad schematic)
At the start: 50 parts, among them Q1 AO3400A, Q10 AO3400A, Q2 AO3400A, Q3 AO3400A, Q4 AO3400A, Q5 AO3400A, Q6 AO3400A, Q7 AO3400A, Q8 AO3400A, Q9 AO3400A

Commit message: Rest of page feedback - Nick
Other:
- note added: "1. Where do Solenoids Connect to? 2. Why is there a voltage divider for the gate of the MOSFET? 3. What interface do we have to connect the solenoids to control board to be driven by MOSFET? 4. Find Flyback diode part and resistor value 5. Break out connectors for each of the solenoids like the net on the left - Nick"
Changed lines of the file:
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@@
 	(generator_version "10.0")
 	(paper "A4")
+	(text "1. Where do Solenoids Connect to? \n2. Why is there a voltage divider for \n	the gate of the MOSFET?\n3. What interface do we have to connect \n	the solenoids to control board \n	to be driven by MOSFET?\n4. Find Flyback diode part and resistor value\n5. Break out connectors for each of the \n	solenoids like the net on the left\n- Nick"
+		(exclude_from_sim no)
+		(at 135.89 39.37 0)
+		(effects
+			(font
+				(size 2.54 2.54)
+				(color 255 0 0 1)
+			)
+			(justify left)
+		)
+	)
 	(junction
 		(at 99.06 100.33)
@@
 		)
 		(stroke
+			(width 0)
+			(type default)
+		)
+	)
+	(wire
+		(pts
+			(xy 99.06 34.29) (xy 128.27 34.29)
+		)
+		(stroke

Commit message: add sam feedback
Other:
- note added: "are L_solenoid the actual solenoids? so this is a low-side switch setup? then those should be Conn_01x02 connectors, not inductor footprints"
Changed lines of the file:
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@@
+		)
+	)
+	(text "are L_solenoid the actual solenoids? so this is a low-side switch setup?\nthen those should be Conn_01x02 connectors, not inductor footprints"
+		(exclude_from_sim no)
+		(at 152.908 123.698 0)
+		(effects
+			(font
+				(size 1.27 1.27)
+			)
 		)
 	)
