File: untitled.kicad_sch (KiCad schematic)
At the start: 10 parts, among them Q1 NMOS, Q10 NMOS, Q2 NMOS, Q3 NMOS, Q4 NMOS, Q5 NMOS, Q6 NMOS, Q7 NMOS, Q8 NMOS, Q9 NMOS

Commit message: Much more progress
hi mom
Parts:
- removed Q1, Q2, Q3, Q4, Q5, Q6, Q7, Q8, Q9: NMOS, symbol Simulation_SPICE:NMOS
- added D10, D11, D12, D3, D4, D5, D6, D7, D8, D9: D, symbol Device:D
- added L1, L10, L2, L3, L4, L5, L6, L7, L8, L9: L_solenoid, symbol Device:L
- added Q11, Q12, Q13, Q14, Q15, Q16, Q17, Q18, Q19: AO3400A, symbol Simulation_SPICE:NMOS
- added R12, R15, R17, R19, R22, R23, R26, R27, R29, R31: 10k, symbol Device:R_US
- added R13, R14, R16, R18, R20, R21, R24, R25, R28, R30: ?????, symbol Device:R_US
- Q10: value NMOS -> AO3400A
Connections:
- net at Q10.1 (D): now also D3.2 (A), L1.2
- net at Q10.2 (G): now also R12.1, R13.2
- net GND: now reaches Q10.3 (S)
- net GND: now also Q11.3 (S), Q12.3 (S), Q13.3 (S), Q14.3 (S), Q15.3 (S), Q16.3 (S), Q17.3 (S), Q18.3 (S), Q19.3 (S), R12.2, R15.2, R17.2, R19.2, R22.2, R23.2, R26.2, R27.2, R29.2, R31.2
- new net: D9.2 (A), L7.2, Q16.1 (D)
- new net: D11.2 (A), L9.2, Q18.1 (D)
- new net: D12.2 (A), L10.2, Q19.1 (D)
- new net: Q15.2 (G), R21.2, R23.1
- new net: Q18.2 (G), R28.2, R29.1
- new net: D8.2 (A), L6.2, Q15.1 (D)
- new net: Q16.2 (G), R24.2, R26.1
- new net: D4.2 (A), L2.2, Q11.1 (D)
- new net: Q11.2 (G), R14.2, R15.1
- new net: Q19.2 (G), R30.2, R31.1
- new net: D5.2 (A), L3.2, Q12.1 (D)
- new net: Q12.2 (G), R16.2, R17.1
- new net: D6.2 (A), L4.2, Q13.1 (D)
- new net: D10.2 (A), L8.2, Q17.1 (D)
- new net: Q17.2 (G), R25.2, R27.1
- new net: D7.2 (A), L5.2, Q14.1 (D)
- new net: Q14.2 (G), R20.2, R22.1
- new net: Q13.2 (G), R18.2, R19.1
- new net 12V: D10.1 (K), D11.1 (K), D12.1 (K), D3.1 (K), D4.1 (K), D5.1 (K), D6.1 (K), D7.1 (K), D8.1 (K), D9.1 (K), L1.1, L10.1, L2.1, L3.1, L4.1, L5.1, L6.1, L7.1, L8.1, L9.1
- new net GATE1: R13.1
- new net GATE10: R30.1
- new net GATE2: R14.1
- new net GATE3: R16.1
- new net GATE4: R18.1
- new net GATE5: R20.1
- new net GATE6: R24.1
- new net GATE7: R21.1
- new net GATE8: R25.1
- new net GATE9: R28.1
Other:
- moved on the sheet: Q10

Commit message: Ok I lied v1 for real
real
Parts:
- renumbered D8 to D10, D10 to D11, D11 to D12, D12 to D13, D3 to D4, D4 to D5, D5 to D6, D6 to D7, D7 to D8, L7 to L6, L6 to L7, Q10 to Q1, Q19 to Q10, Q11 to Q2, Q12 to Q3, Q13 to Q4, Q14 to Q5, Q16 to Q6, Q15 to Q7, Q17 to Q8, Q18 to Q9, R14 to R10, R12 to R11, R15 to R12, R16 to R13, R18 to R14, R17 to R15, R19 to R16, R20 to R17, R24 to R18, R22 to R19, R26 to R20, R25 to R22, R27 to R24, R28 to R25, R30 to R26, R29 to R27, R31 to R28, R13 to R9

Commit message: Commit for Milwaukee Review
Version 0.2 Completed
Parts:
- removed L1, L10, L2, L3, L4, L5, L6, L7, L8, L9: L_solenoid, symbol Device:L
- removed R10, R9: ?????, symbol Device:R_US
- added J10, J11, J12, J13, J14, J15, J16, J17, J8, J9: Conn_01x02, symbol Connector_Generic:Conn_01x02
- added R35, R36: 220, symbol Device:R_US
- R12, R23, R24: value 10k -> 220
- R13, R21, R22: value ????? -> 10k
- R14, R17, R18, R25, R26: value ????? -> 220
Connections:
- net GATE10 is gone; now on net GATE1: R26.1
- net GATE3 is gone; now on net GATE1: R13.1
- net GATE4 is gone; now on net GATE1: R14.1
- net GATE5 is gone; now on net GATE1: R17.1
- net GATE6 is gone; now on net GATE1: R18.1
- net GATE7 is gone; now on net GATE1: R21.1
- net GATE8 is gone; now on net GATE1: R22.1
- net GATE9 is gone; now on net GATE1: R25.1
- net 12V: now also J10.1 (Pin_1), J11.1 (Pin_1), J12.1 (Pin_1), J13.1 (Pin_1), J14.1 (Pin_1), J15.1 (Pin_1), J16.1 (Pin_1), J17.1 (Pin_1), J8.1 (Pin_1), J9.1 (Pin_1)
- net GATE1: now also R11.1, R12.1, R15.1, R16.1, R19.1, R20.1, R23.1, R24.1, R27.1, R28.1, R35.1, R36.1
- net GND: now also R13.2, R21.2, R22.2; no longer R12.2, R23.2, R24.2
- net SOL6_-: now reaches D9.2 (A), Q6.1 (D)
- net SOL6_-: now also J13.2 (Pin_2)
- net SOL9_-: now reaches D12.2 (A), Q9.1 (D)
- net SOL9_-: now also J16.2 (Pin_2)
- net SOL10_-: now reaches D13.2 (A), Q10.1 (D)
- net SOL10_-: now also J17.2 (Pin_2)
- net SOL7_-: now reaches D10.2 (A), Q7.1 (D)
- net SOL7_-: now also J14.2 (Pin_2)
- net SOL2_-: now reaches D5.2 (A), Q2.1 (D)
- net SOL2_-: now also J9.2 (Pin_2)
- net at Q2.2 (G): now also R14.2; no longer R12.1
- net SOL3_-: now reaches D6.2 (A), Q3.1 (D)
- net SOL3_-: now also J10.2 (Pin_2)
- net SOL1_-: now reaches D4.2 (A), Q1.1 (D)
- net SOL1_-: now also J8.2 (Pin_2)
- net SOL4_-: now reaches D7.2 (A), Q4.1 (D)
- net SOL4_-: now also J11.2 (Pin_2)
- net SOL8_-: now reaches D11.2 (A), Q8.1 (D)
- net SOL8_-: now also J15.2 (Pin_2)
- net SOL5_-: now reaches D8.2 (A), Q5.1 (D)
- net SOL5_-: now also J12.2 (Pin_2)
- net at Q1.2 (G): now also R12.2; no longer R11.1
- new net: Q3.2 (G), R17.2
- new net: Q5.2 (G), R23.2
- new net: Q6.2 (G), R24.2
- new net: Q10.2 (G), R36.2
- new net: Q9.2 (G), R35.2
- new net: Q4.2 (G), R18.2
- new net: Q7.2 (G), R25.2
- new net: Q8.2 (G), R26.2

Commit message: Update ig
We messed up
Connections:
- net GATE1: no longer R13.1, R14.1, R15.1, R16.1, R17.1, R18.1, R19.1, R20.1, R21.1, R22.1, R23.1, R24.1, R25.1, R26.1, R27.1, R28.1, R35.1, R36.1
- new net GATE10: R28.1, R36.1
- new net GATE2: R13.1, R14.1
- new net GATE3: R15.1, R17.1
- new net GATE4: R16.1, R18.1
- new net GATE5: R19.1, R23.1
- new net GATE6: R20.1, R24.1
- new net GATE7: R21.1, R25.1
- new net GATE8: R22.1, R26.1
- new net GATE9: R27.1, R35.1

Commit message: 10/14
Fixing my breakout is the only thing... then we can go onto layout
Parts:
- removed Q1, Q10, Q2, Q3, Q4, Q5, Q6, Q7, Q8, Q9: AO3400A, symbol Simulation_SPICE:NMOS
- added Q11, Q12, Q13, Q14, Q15, Q16, Q17, Q18, Q19, Q20: Q_NMOS_GSD, symbol Transistor_FET:Q_NMOS_GSD
Connections:
- net GND: now also Q11.2 (S), Q12.2 (S), Q13.2 (S), Q14.2 (S), Q15.2 (S), Q16.2 (S), Q17.2 (S), Q18.2 (S), Q19.2 (S), Q20.2 (S)
- net SOL10_-: now also Q19.3 (D)
- net SOL1_-: now also Q11.3 (D)
- net SOL2_-: now also Q12.3 (D)
- net SOL3_-: now also Q13.3 (D)
- net SOL4_-: now also Q14.3 (D)
- net SOL5_-: now also Q15.3 (D)
- net SOL6_-: now also Q16.3 (D)
- net SOL7_-: now also Q17.3 (D)
- net SOL8_-: now also Q18.3 (D)
- net SOL9_-: now also Q20.3 (D)
- net at R17.2: now also Q13.1 (G)
- net at R23.2: now also Q15.1 (G)
- net at R24.2: now also Q16.1 (G)
- net at R36.2: now also Q19.1 (G)
- net at R12.2: now also Q11.1 (G)
- net at R35.2: now also Q20.1 (G)
- net at R18.2: now also Q14.1 (G)
- net at R25.2: now also Q17.1 (G)
- net at R26.2: now also Q18.1 (G)
- net at R14.2: now also Q12.1 (G)

Commit message: We are BACK
I am feeling myself. Lots of progress here.
Parts:
- removed J10, J11, J12, J13, J14, J15, J17, J8, J9: Conn_01x02, symbol Connector_Generic:Conn_01x02
- removed R13: 10k, symbol Device:R_US
- added J1, J2, J3, J4: SM02B-GHS-TB, x19_control_library:CONN_SM02B-GHS_JST, symbol Connector_Generic:Conn_01x02
- added J5: SM06B-GHS-TB, x19_control_library:CONN_SM06B-GHS-TB_JST, symbol Connector_Generic:Conn_01x06
- added R12: 10k, Resistor_SMD:R_0603_1608Metric_Pad0.98x0.95mm_HandSolder, symbol Device:R_US
- D10: renamed from D9; value D -> 1N5819HW-7-F; footprint (none) -> x19_control_library:1N5819HW-7-F_DIO
- D11: renamed from D10; value D -> 1N5819HW-7-F; footprint (none) -> x19_control_library:1N5819HW-7-F_DIO
- D12: renamed from D11; value D -> 1N5819HW-7-F; footprint (none) -> x19_control_library:1N5819HW-7-F_DIO
- D13: renamed from D12; value D -> 1N5819HW-7-F; footprint (none) -> x19_control_library:1N5819HW-7-F_DIO
- D14: renamed from D13; value D -> 1N5819HW-7-F; footprint (none) -> x19_control_library:1N5819HW-7-F_DIO
- D5: renamed from D4; value D -> 1N5819HW-7-F; footprint (none) -> x19_control_library:1N5819HW-7-F_DIO
- D6: renamed from D5; value D -> 1N5819HW-7-F; footprint (none) -> x19_control_library:1N5819HW-7-F_DIO
- D7: renamed from D6; value D -> 1N5819HW-7-F; footprint (none) -> x19_control_library:1N5819HW-7-F_DIO
- D8: renamed from D7; value D -> 1N5819HW-7-F; footprint (none) -> x19_control_library:1N5819HW-7-F_DIO
- D9: renamed from D8; value D -> 1N5819HW-7-F; footprint (none) -> x19_control_library:1N5819HW-7-F_DIO
- J6: renamed from J16; value Conn_01x02 -> SM02B-GHS-TB; footprint (none) -> x19_control_library:CONN_SM02B-GHS_JST
- Q1: renamed from Q11; footprint (none) -> x19_control_library:SOT-23-3L_AOS
- Q10: renamed from Q19; footprint (none) -> x19_control_library:SOT-23-3L_AOS
- Q2: renamed from Q12; footprint (none) -> x19_control_library:SOT-23-3L_AOS
- Q3: renamed from Q13; footprint (none) -> x19_control_library:SOT-23-3L_AOS
- Q4: renamed from Q14; footprint (none) -> x19_control_library:SOT-23-3L_AOS
- Q5: renamed from Q15; footprint (none) -> x19_control_library:SOT-23-3L_AOS
- Q6: renamed from Q16; footprint (none) -> x19_control_library:SOT-23-3L_AOS
- Q7: renamed from Q17; footprint (none) -> x19_control_library:SOT-23-3L_AOS
- Q8: renamed from Q18; footprint (none) -> x19_control_library:SOT-23-3L_AOS
- Q9: renamed from Q20; footprint (none) -> x19_control_library:SOT-23-3L_AOS
- R11, R17, R18, R19, R20, R21, R22, R23, R24, R25, R26, R27, R28: footprint (none) -> Resistor_SMD:R_0603_1608Metric_Pad0.98x0.95mm_HandSolder
- R13: renamed from R15; footprint (none) -> Resistor_SMD:R_0603_1608Metric_Pad0.98x0.95mm_HandSolder
- R14: renamed from R16; footprint (none) -> Resistor_SMD:R_0603_1608Metric_Pad0.98x0.95mm_HandSolder
- R15: renamed from R12; footprint (none) -> Resistor_SMD:R_0603_1608Metric_Pad0.98x0.95mm_HandSolder
- R16: renamed from R14; footprint (none) -> Resistor_SMD:R_0603_1608Metric_Pad0.98x0.95mm_HandSolder
- R29: renamed from R35; footprint (none) -> Resistor_SMD:R_0603_1608Metric_Pad0.98x0.95mm_HandSolder
- R30: renamed from R36; footprint (none) -> Resistor_SMD:R_0603_1608Metric_Pad0.98x0.95mm_HandSolder
Connections:
- net 12V: now also J5.1 (Pin_1), J5.2 (Pin_2), J5.3 (Pin_3), J5.4 (Pin_4), J5.5 (Pin_5), J5.6 (Pin_6); no longer J6.1 (Pin_1)
- net GND: now also R12.2
- net GATE1 renamed SOL1A
- net GATE10 renamed SOL5B
- net GATE2 renamed SOL1B
- net SOL1B: now also R12.1
- net GATE3 renamed SOL2A
- net GATE4 renamed SOL2B
- net GATE5 renamed SOL3A
- net GATE6 renamed SOL3B
- net GATE7 renamed SOL4A
- net GATE8 renamed SOL4B
- net GATE9 renamed SOL5A
- net SOL10_- renamed SOL5B-
- net SOL5B-: now also J6.2 (Pin_2)
- net SOL1_- renamed SOL1A-
- net SOL1A-: now also J2.1 (Pin_1)
- net SOL2_- renamed SOL1B-
- net SOL1B-: now also J2.2 (Pin_2)
- net SOL3_- renamed SOL2A-
- net SOL2A-: now also J1.1 (Pin_1)
- net SOL4_- renamed SOL2B-
- net SOL2B-: now also J1.2 (Pin_2)
- net SOL5_- renamed SOL3A-
- net SOL3A-: now also J3.1 (Pin_1)
- net SOL6_- renamed SOL3B-
- net SOL3B-: now also J3.2 (Pin_2)
- net SOL7_- renamed SOL4A-
- net SOL4A-: now also J4.1 (Pin_1)
- net SOL8_- renamed SOL4B-
- net SOL4B-: now also J4.2 (Pin_2)
- net SOL9_- renamed SOL5A-
- net SOL5A-: now also J6.1 (Pin_1); no longer J6.2 (Pin_2)
Other:
- note added: "Signal GND Power Signal"
- moved on the sheet: J6
