File: untitled.kicad_sch (KiCad schematic)
At the start: 46 parts, among them J1 SM02B-GHS-TB, J2 SM02B-GHS-TB, J3 SM02B-GHS-TB, J4 SM02B-GHS-TB, J5 SM06B-GHS-TB, J6 SM02B-GHS-TB, Q1 Q_NMOS_GSD, Q10 Q_NMOS_GSD, Q2 Q_NMOS_GSD, Q3 Q_NMOS_GSD, Q4 Q_NMOS_GSD, Q5 Q_NMOS_GSD, Q6 Q_NMOS_GSD, Q7 Q_NMOS_GSD, Q8 Q_NMOS_GSD, Q9 Q_NMOS_GSD

Commit message: Sized
bang
Parts:
- J1, J2, J3, J4, J6: footprint x19_control_library:CONN_SM02B-GHS_JST -> x19_control_library:CONN_SM02B-GHS_JST_solder_joint
- J5: footprint x19_control_library:CONN_SM06B-GHS-TB_JST -> x19_control_library:CONN_SM06B-GHS-TB_JST_solder_joint
- renumbered R11 to R10, R12 to R11, R13 to R12, R14 to R13, R15 to R14, R16 to R15, R17 to R16, R18 to R17, R19 to R18, R20 to R19, R21 to R20, R22 to R21, R23 to R22, R24 to R23, R25 to R24, R26 to R25, R27 to R26, R28 to R27, R29 to R28, R30 to R29

Commit message: Update update 10/28
(It rhymes)
Parts:
- R19: value 10k -> 4.7k
Other:
- note added: "3 is the backup"
Changed lines of the file:
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@@
 	(generator_version "10.0")
 	(paper "A4")
+	(text "3 is the backup"
+		(exclude_from_sim no)
+		(at 99.568 6.858 0)
+		(effects
+			(font
+				(size 1.27 1.27)
+				(color 254 90 255 1)
+			)
+		)
+	)
 	(text "Signal\nGND\nPower\nSignal\n"
 		(exclude_from_sim no)
@@
 			)
 		)
-		(property "Value" "10k"
+		(property "Value" "4.7k"
 			(at 124.46 90.1699 0)
 			(show_name no)

Commit message: Layout Placement Is Happening
The other members are CHUD rn
Parts:
- J1, J2, J3, J4, J6: footprint x19_control_library:CONN_SM02B-GHS_JST_solder_joint -> x19_control_library:Vertical_CONN_BM02B-GHS-TBT_JST
- J5: footprint x19_control_library:CONN_SM06B-GHS-TB_JST_solder_joint -> x19_control_library:vertical_CONN_BM06B-GHS-TBT_JST
- renumbered R10 to R11, R11 to R12, R12 to R13, R13 to R14, R14 to R15, R15 to R16, R16 to R17, R17 to R18, R18 to R19, R19 to R20, R20 to R21, R21 to R22, R22 to R23, R23 to R24, R24 to R25, R25 to R26, R26 to R27, R27 to R28, R28 to R29, R29 to R30
