File: Power_Monitoring.kicad_sch (KiCad schematic)
At the start: 10 parts, among them U5 INA237AIDGSR, U7 INA237AIDGSR

Commit message: Commit for Milwaukee Review
Version 0.2 Completed
Parts:
- removed C12, C13: 0.1u, symbol Device:C
- removed C14, C15: C, symbol Device:C
- removed R10, R8: 10k, symbol Device:R_US
- removed R11: 120m, symbol Device:R_Shunt_US
- removed R9: 15m, symbol Device:R_Shunt_US
- removed U5, U7: INA237AIDGSR, VSSOP_IDGSR_TEX, symbol board_control_manual_lib:INA237AIDGSR
Other:
- note removed: "I2C Connect"
- note removed: "R_pu"
- note removed: "Said via"
- note removed: "Said vias"
