File: X19-Control-Board.kicad_pcb (KiCad board)
At the start: 4 copper layers, 56.9 x 119.5 mm, 0 parts

Commit message: Sized
bang
Parts:
- added C1: 2.2u, Capacitor_SMD:C_0603_1608Metric_Pad1.08x0.95mm_HandSolder, F.Cu at (106.6, 19.8)
- added C10: 0.1u, Capacitor_SMD:C_0603_1608Metric_Pad1.08x0.95mm_HandSolder, F.Cu at (111.0, 29.8)
- added C11: 0.1u, Capacitor_SMD:C_0603_1608Metric_Pad1.08x0.95mm_HandSolder, F.Cu at (115.3, 19.8)
- added C12: 0.1u, Capacitor_SMD:C_0603_1608Metric_Pad1.08x0.95mm_HandSolder, F.Cu at (75.5, 54.6)
- added C13: 0.1u, Capacitor_SMD:C_0603_1608Metric_Pad1.08x0.95mm_HandSolder, F.Cu at (75.5, 57.1)
- added C14: 0.1u, Capacitor_SMD:C_0603_1608Metric_Pad1.08x0.95mm_HandSolder, F.Cu at (106.6, 54.5)
- added C15: 0.1u, Capacitor_SMD:C_0603_1608Metric_Pad1.08x0.95mm_HandSolder, F.Cu at (106.6, 57.0)
- added C16: 1u, Capacitor_SMD:C_0603_1608Metric_Pad1.08x0.95mm_HandSolder, F.Cu at (106.6, 59.5)
- added C17: 1u, Capacitor_SMD:C_0603_1608Metric_Pad1.08x0.95mm_HandSolder, F.Cu at (106.6, 62.0)
- added C2: 0.1u, Capacitor_SMD:C_0603_1608Metric_Pad1.08x0.95mm_HandSolder, F.Cu at (106.6, 22.3)
- added C3: 0.1u, Capacitor_SMD:C_0603_1608Metric_Pad1.08x0.95mm_HandSolder, F.Cu at (106.6, 24.8)
- added C4: 0.1u, Capacitor_SMD:C_0603_1608Metric_Pad1.08x0.95mm_HandSolder, F.Cu at (106.6, 27.3)
- added C5: 0.1u, Capacitor_SMD:C_0603_1608Metric_Pad1.08x0.95mm_HandSolder, F.Cu at (106.6, 29.8)
- added C6: 4.7u, Capacitor_SMD:C_0603_1608Metric_Pad1.08x0.95mm_HandSolder, F.Cu at (111.0, 19.8)
- added C7: 8p, Capacitor_SMD:C_0603_1608Metric_Pad1.08x0.95mm_HandSolder, F.Cu at (111.0, 22.3)
- added C8: 8p, Capacitor_SMD:C_0603_1608Metric_Pad1.08x0.95mm_HandSolder, F.Cu at (111.0, 24.8)
- added C9: 0.1u, Capacitor_SMD:C_0603_1608Metric_Pad1.08x0.95mm_HandSolder, F.Cu at (111.0, 27.3)
- added CR1: ESD2CAN24DBZRQ1, x19_control_library:ESD2CAN24DBZRQ1, F.Cu at (42.1, 60.2)
- added D1: ORANGE, x19_control_library:LTST-C191KFKT_1_anode_2_cathode, F.Cu at (123.7, 32.3)
- added D10: 1N5819HW-7-F, x19_control_library:1N5819HW-7-F_DIO, F.Cu at (75.6, 37.0)
- added D11: 1N5819HW-7-F, x19_control_library:1N5819HW-7-F_DIO, F.Cu at (75.6, 40.3)
- added D12: 1N5819HW-7-F, x19_control_library:1N5819HW-7-F_DIO, F.Cu at (75.6, 43.7)
- added D13: 1N5819HW-7-F, x19_control_library:1N5819HW-7-F_DIO, F.Cu at (75.6, 47.1)
- added D14: 1N5819HW-7-F, x19_control_library:1N5819HW-7-F_DIO, F.Cu at (75.6, 50.4)
- added D2: BLUE, x19_control_library:LTST-C191KFKT_1_anode_2_cathode, F.Cu at (123.7, 34.8)
- added D3: GREEN, x19_control_library:LTST-C191KFKT_1_anode_2_cathode, F.Cu at (123.7, 37.2)
- added D4: RED, x19_control_library:LTST-C191KFKT_1_anode_2_cathode, F.Cu at (123.7, 39.7)
- added D5: 1N5819HW-7-F, x19_control_library:1N5819HW-7-F_DIO, F.Cu at (75.6, 20.2)
- added D6: 1N5819HW-7-F, x19_control_library:1N5819HW-7-F_DIO, F.Cu at (75.6, 23.5)
- added D7: 1N5819HW-7-F, x19_control_library:1N5819HW-7-F_DIO, F.Cu at (75.6, 26.9)
- added D8: 1N5819HW-7-F, x19_control_library:1N5819HW-7-F_DIO, F.Cu at (75.6, 30.3)
- added D9: 1N5819HW-7-F, x19_control_library:1N5819HW-7-F_DIO, F.Cu at (75.6, 33.6)
- added J1: SM02B-GHS-TB, x19_control_library:CONN_SM02B-GHS_JST_solder_joint, F.Cu at (20.5, 84.8)
- added J10: IPS1-105-01-L-D, x19_control_library:SAMTEC_IPS1-105-01-S-D, F.Cu at (41.9, 22.4)
- added J11: 61300511821, x19_control_library:61300511821, F.Cu at (20.4, 99.9)
- added J12: 61300511821, x19_control_library:61300511821, F.Cu at (58.2, 79.4)
- added J2: SM02B-GHS-TB, x19_control_library:CONN_SM02B-GHS_JST_solder_joint, F.Cu at (21.7, 65.2)
- added J3: SM02B-GHS-TB, x19_control_library:CONN_SM02B-GHS_JST_solder_joint, F.Cu at (20.4, 74.4)
- added J4: SM02B-GHS-TB, x19_control_library:CONN_SM02B-GHS_JST_solder_joint, F.Cu at (21.7, 53.9)
- added J5: SM06B-GHS-TB, x19_control_library:CONN_SM06B-GHS-TB_JST_solder_joint, F.Cu at (25.1, 27.7)
- added J6: SM02B-GHS-TB, x19_control_library:CONN_SM02B-GHS_JST_solder_joint, F.Cu at (22.8, 43.0)
- added J7: SM04B-GHS-TB, x19_control_library:CONN_BM04B-GHS-TBT_JST_solder_joint, F.Cu at (43.7, 104.9)
- added J8: 6 pin one, Connector_PinHeader_2.54mm:PinHeader_1x06_P2.54mm_Vertical, F.Cu at (68.8, 114.6)
- added J9: 6 pin one, Connector_PinHeader_2.54mm:PinHeader_1x06_P2.54mm_Vertical, F.Cu at (60.4, 114.7)
- added Q1: Q_NMOS_GSD, x19_control_library:SOT-23-3L_AOS, F.Cu at (81.0, 21.2)
- added Q10: Q_NMOS_GSD, x19_control_library:SOT-23-3L_AOS, F.Cu at (100.1, 26.5)
- added Q2: Q_NMOS_GSD, x19_control_library:SOT-23-3L_AOS, F.Cu at (85.8, 21.2)
- added Q3: Q_NMOS_GSD, x19_control_library:SOT-23-3L_AOS, F.Cu at (90.6, 21.2)
- added Q4: Q_NMOS_GSD, x19_control_library:SOT-23-3L_AOS, F.Cu at (95.3, 21.2)
- added Q5: Q_NMOS_GSD, x19_control_library:SOT-23-3L_AOS, F.Cu at (100.1, 21.2)
- added Q6: Q_NMOS_GSD, x19_control_library:SOT-23-3L_AOS, F.Cu at (81.0, 26.5)
- added Q7: Q_NMOS_GSD, x19_control_library:SOT-23-3L_AOS, F.Cu at (85.8, 26.5)
- added Q8: Q_NMOS_GSD, x19_control_library:SOT-23-3L_AOS, F.Cu at (90.6, 26.5)
- added Q9: Q_NMOS_GSD, x19_control_library:SOT-23-3L_AOS, F.Cu at (95.3, 26.5)
- added R1: 10k, Resistor_SMD:R_0603_1608Metric_Pad0.98x0.95mm_HandSolder, F.Cu at (115.3, 22.3)
- added R10: 10k, Resistor_SMD:R_0603_1608Metric_Pad0.98x0.95mm_HandSolder, F.Cu at (80.8, 30.5)
- added R11: 10k, Resistor_SMD:R_0603_1608Metric_Pad0.98x0.95mm_HandSolder, F.Cu at (80.8, 33.0)
- added R12: 10k, Resistor_SMD:R_0603_1608Metric_Pad0.98x0.95mm_HandSolder, F.Cu at (80.8, 35.5)
- added R13: 10k, Resistor_SMD:R_0603_1608Metric_Pad0.98x0.95mm_HandSolder, F.Cu at (80.8, 38.0)
- added R14: 220, Resistor_SMD:R_0603_1608Metric_Pad0.98x0.95mm_HandSolder, F.Cu at (80.8, 40.5)
- added R15: 220, Resistor_SMD:R_0603_1608Metric_Pad0.98x0.95mm_HandSolder, F.Cu at (85.2, 30.5)
- added R16: 220, Resistor_SMD:R_0603_1608Metric_Pad0.98x0.95mm_HandSolder, F.Cu at (85.2, 33.0)
- added R17: 220, Resistor_SMD:R_0603_1608Metric_Pad0.98x0.95mm_HandSolder, F.Cu at (85.2, 35.5)
- added R18: 10k, Resistor_SMD:R_0603_1608Metric_Pad0.98x0.95mm_HandSolder, F.Cu at (85.2, 38.0)
- added R19: 10k, Resistor_SMD:R_0603_1608Metric_Pad0.98x0.95mm_HandSolder, F.Cu at (85.2, 40.5)
- added R2: 0, Resistor_SMD:R_0603_1608Metric_Pad0.98x0.95mm_HandSolder, F.Cu at (115.3, 24.8)
- added R20: 10k, Resistor_SMD:R_0603_1608Metric_Pad0.98x0.95mm_HandSolder, F.Cu at (89.5, 30.5)
- added R21: 10k, Resistor_SMD:R_0603_1608Metric_Pad0.98x0.95mm_HandSolder, F.Cu at (89.5, 33.0)
- added R22: 220, Resistor_SMD:R_0603_1608Metric_Pad0.98x0.95mm_HandSolder, F.Cu at (89.5, 35.5)
- added R23: 220, Resistor_SMD:R_0603_1608Metric_Pad0.98x0.95mm_HandSolder, F.Cu at (89.5, 38.0)
- added R24: 220, Resistor_SMD:R_0603_1608Metric_Pad0.98x0.95mm_HandSolder, F.Cu at (89.5, 40.5)
- added R25: 220, Resistor_SMD:R_0603_1608Metric_Pad0.98x0.95mm_HandSolder, F.Cu at (93.9, 30.5)
- added R26: 10k, Resistor_SMD:R_0603_1608Metric_Pad0.98x0.95mm_HandSolder, F.Cu at (93.9, 33.0)
- added R27: 10k, Resistor_SMD:R_0603_1608Metric_Pad0.98x0.95mm_HandSolder, F.Cu at (93.9, 35.5)
- added R28: 220, Resistor_SMD:R_0603_1608Metric_Pad0.98x0.95mm_HandSolder, F.Cu at (93.9, 38.0)
- added R29: 220, Resistor_SMD:R_0603_1608Metric_Pad0.98x0.95mm_HandSolder, F.Cu at (93.9, 40.5)
- added R3: 60, Resistor_SMD:R_0603_1608Metric_Pad0.98x0.95mm_HandSolder, F.Cu at (115.3, 27.3)
- added R30: 10k, Resistor_SMD:R_0603_1608Metric_Pad0.98x0.95mm_HandSolder, F.Cu at (106.6, 64.5)
- added R31: 10k, Resistor_SMD:R_0603_1608Metric_Pad0.98x0.95mm_HandSolder, F.Cu at (106.6, 67.0)
- added R32: 10k, Resistor_SMD:R_0603_1608Metric_Pad0.98x0.95mm_HandSolder, F.Cu at (106.6, 69.6)
- added R33: 1m, Resistor_SMD:R_0603_1608Metric_Pad0.98x0.95mm_HandSolder, F.Cu at (106.6, 72.1)
- added R34: 1m, Resistor_SMD:R_0603_1608Metric_Pad0.98x0.95mm_HandSolder, F.Cu at (106.6, 74.6)
- added R4: 60, Resistor_SMD:R_0603_1608Metric_Pad0.98x0.95mm_HandSolder, F.Cu at (115.3, 29.8)
- added R5: 10k, Resistor_SMD:R_0603_1608Metric_Pad0.98x0.95mm_HandSolder, F.Cu at (119.7, 19.8)
- added R6: 120, Resistor_SMD:R_0603_1608Metric_Pad0.98x0.95mm_HandSolder, F.Cu at (119.7, 22.3)
- added R7: 1k, Resistor_SMD:R_0603_1608Metric_Pad0.98x0.95mm_HandSolder, F.Cu at (119.7, 24.8)
- added R8: 120, Resistor_SMD:R_0603_1608Metric_Pad0.98x0.95mm_HandSolder, F.Cu at (119.7, 27.3)
- added R9: 120, Resistor_SMD:R_0603_1608Metric_Pad0.98x0.95mm_HandSolder, F.Cu at (119.7, 29.8)
- added TP1: GND_TP, TestPoint:TestPoint_Pad_D3.0mm, F.Cu at (107.0, 33.6)
- added TP2: 5.2V_TP, TestPoint:TestPoint_Pad_D3.0mm, F.Cu at (107.0, 38.6)
- added TP3: 12V_TP, TestPoint:TestPoint_Pad_D3.0mm, F.Cu at (107.0, 43.7)
- added TP4: 3.3VTP, TestPoint:TestPoint_Pad_D3.0mm, F.Cu at (107.0, 48.7)
- added U1: TCAN1044AEVDRQ1, x19_control_library:TCAN1044AEVDRQ1, F.Cu at (42.1, 66.8)
- added U2: STM32C542CCT6, x19_control_library:STM32C542CCT6, F.Cu at (42.5, 79.4)
- added U3: BMI270, x19_control_library:BMI270_BOS, F.Cu at (45.9, 119.6)
- added U4: INA237AIDGSR, x19_control_library:INA237AIDGSR, F.Cu at (50.3, 127.8)
- added U5: INA237AIDGSR, x19_control_library:INA237AIDGSR, F.Cu at (40.8, 128.5)
- added U6: MIC5504-3.3YM5-TR, x19_control_library:MIC5504_3_3YM5_TR, F.Cu at (33.4, 88.0)
- added Y1: ECS-240-8-37B-CKY-TR, x19_control_library:ECS-240-8-37CKM_ECS, F.Cu at (33.4, 79.6)
Other:
- board size 56.9 x 119.5 mm -> 57 x 119.5 mm
- board text added: "These need to be spaced carefully, consider a new footprint that puts them together"

Commit message: Layout Placement Is Happening
The other members are CHUD rn
Parts:
- removed J8, J9: 6 pin one, Connector_PinHeader_2.54mm:PinHeader_1x06_P2.54mm_Vertical
- added C18: 0.1u, Capacitor_SMD:C_0603_1608Metric_Pad1.08x0.95mm_HandSolder, F.Cu at (64.3, 56.4)
- added C19: 1u, Capacitor_SMD:C_0603_1608Metric_Pad1.08x0.95mm_HandSolder, F.Cu at (64.3, 59.0)
- added C20: 1u, Capacitor_SMD:C_0603_1608Metric_Pad1.08x0.95mm_HandSolder, F.Cu at (64.3, 61.5)
- added J13: Conn_01x03_Socket, Connector_PinHeader_2.54mm:PinHeader_1x03_P2.54mm_Vertical, F.Cu at (26.9, 111.0)
- added J14: Conn_01x03_Socket, Connector_PinHeader_2.54mm:PinHeader_1x03_P2.54mm_Vertical, F.Cu at (31.5, 111.0)
- added J15: Conn_01x03_Socket, Connector_PinHeader_2.54mm:PinHeader_1x03_P2.54mm_Vertical, F.Cu at (36.1, 111.0)
- added J16: Conn_01x03_Socket, Connector_PinHeader_2.54mm:PinHeader_1x03_P2.54mm_Vertical, F.Cu at (40.7, 111.0)
- added J17: Conn_01x03_Socket, Connector_PinHeader_2.54mm:PinHeader_1x03_P2.54mm_Vertical, F.Cu at (45.3, 111.0)
- added J18: IPS1-105-01-L-D, x19_control_library:SAMTEC_IPS1-105-01-S-D, F.Cu at (3.05, 77.0)
- added J19: 61300511821, x19_control_library:61300511821, F.Cu at (3.05, 109.2)
- added J20: 61300511821, x19_control_library:61300511821, F.Cu at (3.05, 93.2)
- added U7: ~, x19_control_library:MODULE_4754, F.Cu at (44.2, 91.2)
- C12, C13, C14: value 0.1u -> 22u; footprint Capacitor_SMD:C_0603_1608Metric_Pad1.08x0.95mm_HandSolder -> Capacitor_SMD:C_1206_3216Metric_Pad1.33x1.80mm_HandSolder
- C16, C17: value 1u -> 0.1u
- J1, J2, J3, J4, J6: footprint x19_control_library:CONN_SM02B-GHS_JST_solder_joint -> x19_control_library:Vertical_CONN_BM02B-GHS-TBT_JST
- J10: value IPS1-105-01-L-D -> Conn_01x03_Socket; footprint x19_control_library:SAMTEC_IPS1-105-01-S-D -> Connector_PinHeader_2.54mm:PinHeader_1x03_P2.54mm_Vertical
- J11, J12: value 61300511821 -> Conn_01x03_Socket; footprint x19_control_library:61300511821 -> Connector_PinHeader_2.54mm:PinHeader_1x03_P2.54mm_Vertical
- J5: footprint x19_control_library:CONN_SM06B-GHS-TB_JST_solder_joint -> x19_control_library:vertical_CONN_BM06B-GHS-TBT_JST
- J7: footprint x19_control_library:CONN_BM04B-GHS-TBT_JST_solder_joint -> x19_control_library:vertical_CONN_BM04B-GHS-TBT_JST
- R10: value 10k -> 120
- R14, R22, R28: value 220 -> 10k
- R18, R26, R30: value 10k -> 220
- R20: value 10k -> 4.7k
- R33: value 1m -> 100m
- R34: value 1m -> 5m
- R6: value 120 -> 10k
- R7: value 1k -> 120
- R8: value 120 -> 1k
- moved J10 93.1 mm to (13.2, 111.0)
- moved R5 90.3 mm to (72.3, 96.6)
- moved J1 84.6 mm to (53.3, 6.86), turned to 90 degrees
- moved C15 84.1 mm to (30.1, 91.9)
- moved C16 84.1 mm to (30.1, 94.4)
- moved C6 83.7 mm to (68.0, 91.6)
- moved C7 83.7 mm to (68.0, 94.1)
- moved C8 83.7 mm to (68.0, 96.6)
- moved C11 77.4 mm to (72.3, 84.0)
- moved R1 77.4 mm to (72.3, 86.6)
- moved R2 77.4 mm to (72.3, 89.1)
- moved R3 77.4 mm to (72.3, 91.6)
- moved R4 77.4 mm to (72.3, 94.1)
- moved TP4 77.3 mm to (77.2, 120.1)
- moved TP1 77.3 mm to (77.2, 104.9)
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Connections:
- net INT1_BOTH_IMU renamed INT_BMI
- C1 pad 1: 3.3V -> Net-(U2-VCAP)
- C12 pad 1: 3.3V -> 5.2V
- C13 pad 1: 3.3V -> 12V
- C14 pad 1: 3.3V -> 12V
- C16 pad 1: 5.2V -> 3.3V
- J11 pad 1: nRST -> GND
- J11 pad 2: SWCLK -> unconnected-(J11-Pin_2-Pad2)
- J11 pad 3: SWDIO -> PWM2
- J12 pad 1: CAN_H -> GND
- J12 pad 2: CAN_L -> unconnected-(J12-Pin_2-Pad2)
- J12 pad 3: MOSI -> PWM3
- R10 pad 1: SOL1A -> Net-(D4-K)
- R11 pad 1: SOL1B -> SOL1A
- R12 pad 1: SOL2A -> SOL1B
- R13 pad 1: SOL2B -> SOL2A
- R14 pad 1: SOL1A -> SOL2B
- R14 pad 2: Net-(Q1-G) -> GND
- R15 pad 1: SOL1B -> SOL1A
- R15 pad 2: Net-(Q2-G) -> Net-(Q1-G)
- R16 pad 1: SOL2A -> SOL1B
- R16 pad 2: Net-(Q3-G) -> Net-(Q2-G)
- R17 pad 1: SOL2B -> SOL2A
- R17 pad 2: Net-(Q4-G) -> Net-(Q3-G)
- R18 pad 1: SOL3A -> SOL2B
- R18 pad 2: GND -> Net-(Q4-G)
- R19 pad 1: SOL3B -> SOL3A
- R20 pad 1: SOL4A -> SOL3B
- R21 pad 1: SOL4B -> SOL4A
- R22 pad 1: SOL3A -> SOL4B
- R22 pad 2: Net-(Q5-G) -> GND
- R23 pad 1: SOL3B -> SOL3A
- R23 pad 2: Net-(Q6-G) -> Net-(Q5-G)
- R24 pad 1: SOL4A -> SOL3B
- R24 pad 2: Net-(Q7-G) -> Net-(Q6-G)
- R25 pad 1: SOL4B -> SOL4A
- R25 pad 2: Net-(Q8-G) -> Net-(Q7-G)
- R26 pad 1: SOL5A -> SOL4B
- R26 pad 2: GND -> Net-(Q8-G)
- R27 pad 1: SOL5B -> SOL5A
- R28 pad 1: SOL5A -> SOL5B
- R28 pad 2: Net-(Q9-G) -> GND
- R29 pad 1: SOL5B -> SOL5A
- R29 pad 2: Net-(Q10-G) -> Net-(Q9-G)
- R30 pad 1: 3.3V -> SOL5B
- R30 pad 2: 5.2V_ALERT -> Net-(Q10-G)
- R31 pad 2: 12V_ALERT -> 5.2V_ALERT
- R32 pad 2: Net-(U5-A0) -> 12V_ALERT
- R5 pad 1: 3.3V -> Net-(U2-PH2-BOOT0)
- R5 pad 2: SDA -> GND
- R6 pad 1: Net-(D1-K) -> 3.3V
- R6 pad 2: GND -> SDA
- R7 pad 1: Net-(D2-K) -> Net-(D1-K)
- R8 pad 1: Net-(D3-K) -> Net-(D2-K)
- R9 pad 1: Net-(D4-K) -> Net-(D3-K)
- U1 pad 1: STM_TO_INPUT_CAN -> CAN_TX
- U1 pad 4: STM_TO_OUTPUT_CAN -> CAN_RX
- U2 pad 2: unconnected-(U2-PC13-Pad2) -> INT_BN0
- U2 pad 22: 3.3V -> Net-(U2-VCAP)
- U2 pad 43: STM_TO_OUTPUT_CAN -> CAN_TX
- U2 pad 44: unconnected-(U2-PH2-BOOT0-Pad44) -> Net-(U2-PH2-BOOT0)
- U2 pad 45: STM_TO_INPUT_CAN -> CAN_RX
- U5 pad 2: Net-(U5-A0) -> 3.3V
Other:
- board text removed: "Check board Dim"
